File: Schamatic/Motor/V3/v3.sch (KiCad schematic (older format))
At the start: 30 parts, among them J1 SWD, J2 SENSOR, J3 CAN, Q1 PSMN3R3-40YS, Q2 PSMN3R3-40YS, Q3 PSMN3R3-40YS, Q4 PSMN3R3-40YS, Q5 PSMN3R3-40YS, Q6 PSMN3R3-40YS, U1 STSPIN32F0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

Commit message: new version of controller
Parts:
- added J10: U, symbol CONN_01X01
- added J11: W, symbol CONN_01X01
- added J12: V, symbol CONN_01X01
- added J4, J5, J6: 12, symbol CONN_01X01
- added J7, J8, J9: GND, symbol CONN_01X01
Changed lines of the file:
@@
 LIBS:contrib
 LIBS:valves
-LIBS:Misha
 LIBS:v3-cache
 EELAYER 25 0
@@
 	0    -1   -1   0
 $EndComp
+$Comp
+L CONN_01X01 J10
+U 1 1 59CA3A1D
+P 8000 2100
+F 0 "J10" H 8000 2200 50  0000 C CNN
+F 1 "U" V 8100 2100 50  0000 C CNN
+F 2 "" H 8000 2100 50  0001 C CNN
+F 3 "" H 8000 2100 50  0001 C CNN
+	1    8000 2100
+	1    0    0    -1
+$EndComp
+$Comp
+L CONN_01X01 J11
+U 1 1 59CA3AAA
+P 8000 3550
+F 0 "J11" H 8000 3650 50  0000 C CNN
+F 1 "W" V 8100 3550 50  0000 C CNN
+F 2 "" H 8000 3550 50  0001 C CNN
+F 3 "" H 8000 3550 50  0001 C CNN
+	1    8000 3550
+	1    0    0    -1
+$EndComp
+$Comp
+L CONN_01X01 J12
+U 1 1 59CA3B19
+P 8000 4900
+F 0 "J12" H 8000 5000 50  0000 C CNN
+F 1 "V" V 8100 4900 50  0000 C CNN
+F 2 "" H 8000 4900 50  0001 C CNN
+F 3 "" H 8000 4900 50  0001 C CNN
+	1    8000 4900
+	1    0    0    -1
+$EndComp
+$Comp
+L CONN_01X01 J6
+U 1 1 59CA46E3
+P 1050 6750
+F 0 "J6" H 1050 6850 50  0000 C CNN
+F 1 "12" V 1150 6750 50  0000 C CNN
+F 2 "" H 1050 6750 50  0001 C CNN
+F 3 "" H 1050 6750 50  0001 C CNN
+	1    1050 6750
+	-1   0    0    1
+$EndComp
+$Comp
+L CONN_01X01 J5
+U 1 1 59CA474E
+P 1050 6600
+F 0 "J5" H 1050 6700 50  0000 C CNN
+F 1 "12" V 1150 6600 50  0000 C CNN
+F 2 "" H 1050 6600 50  0001 C CNN
+F 3 "" H 1050 6600 50  0001 C CNN
+	1    1050 6600
+	-1   0    0    1
+$EndComp
+$Comp
+L CONN_01X01 J4
+U 1 1 59CA47AD
+P 1050 6450
+F 0 "J4" H 1050 6550 50  0000 C CNN
+F 1 "12" V 1150 6450 50  0000 C CNN
+F 2 "" H 1050 6450 50  0001 C CNN
+F 3 "" H 1050 6450 50  0001 C CNN
+	1    1050 6450
+	-1   0    0    1
+$EndComp
+$Comp
+L +12V #PWR027
+U 1 1 59CA4F88
+P 1250 6450
+F 0 "#PWR027" H 1250 6300 50  0001 C CNN
+F 1 "+12V" H 1250 6590 50  0000 C CNN
+F 2 "" H 1250 6450 50  0001 C CNN
+F 3 "" H 1250 6450 50  0001 C CNN
+	1    1250 6450
+	0    1    1    0
+$EndComp
+$Comp
+L +12V #PWR028
+U 1 1 59CA5230
+P 1250 6600
+F 0 "#PWR028" H 1250 6450 50  0001 C CNN
+F 1 "+12V" H 1250 6740 50  0000 C CNN
+F 2 "" H 1250 6600 50  0001 C CNN
+F 3 "" H 1250 6600 50  0001 C CNN
+	1    1250 6600
+	0    1    1    0
+$EndComp
+$Comp
+L +12V #PWR029
+U 1 1 59CA52B0
+P 1250 6750
+F 0 "#PWR029" H 1250 6600 50  0001 C CNN
+F 1 "+12V" H 1250 6890 50  0000 C CNN
+F 2 "" H 1250 6750 50  0001 C CNN
+F 3 "" H 1250 6750 50  0001 C CNN
+	1    1250 6750
+	0    1    1    0
+$EndComp
+$Comp
+L CONN_01X01 J9
+U 1 1 59CA54D7
+P 1050 7400
+F 0 "J9" H 1050 7500 50  0000 C CNN
+F 1 "GND" V 1150 7400 50  0000 C CNN
+F 2 "" H 1050 7400 50  0001 C CNN
+F 3 "" H 1050 7400 50  0001 C CNN
+	1    1050 7400
+	-1   0    0    1
+$EndComp
+$Comp
+L CONN_01X01 J8
+U 1 1 59CA54DE
+P 1050 7250
+F 0 "J8" H 1050 7350 50  0000 C CNN
+F 1 "GND" V 1150 7250 50  0000 C CNN
+F 2 "" H 1050 7250 50  0001 C CNN
+F 3 "" H 1050 7250 50  0001 C CNN
+	1    1050 7250
+	-1   0    0    1
+$EndComp
+$Comp
+L CONN_01X01 J7
+U 1 1 59CA54E5
+P 1050 7100
+F 0 "J7" H 1050 7200 50  0000 C CNN
+F 1 "GND" V 1150 7100 50  0000 C CNN
+F 2 "" H 1050 7100 50  0001 C CNN
+F 3 "" H 1050 7100 50  0001 C CNN
+	1    1050 7100
+	-1   0    0    1
+$EndComp
+$Comp
+L Earth #PWR030
+U 1 1 59CA564E
+P 1250 7100
+F 0 "#PWR030" H 1250 6850 50  0001 C CNN
+F 1 "Earth" H 1250 6950 50  0001 C CNN
+F 2 "" H 1250 7100 50  0001 C CNN
+F 3 "" H 1250 7100 50  0001 C CNN
+	1    1250 7100
+	0    -1   -1   0
+$EndComp
+$Comp
+L Earth #PWR031
+U 1 1 59CA56CE
+P 1250 7250
+F 0 "#PWR031" H 1250 7000 50  0001 C CNN
+F 1 "Earth" H 1250 7100 50  0001 C CNN
+F 2 "" H 1250 7250 50  0001 C CNN
+F 3 "" H 1250 7250 50  0001 C CNN
+	1    1250 7250
+	0    -1   -1   0
+$EndComp
+$Comp
+L Earth #PWR032
+U 1 1 59CA574E
+P 1250 7400
+F 0 "#PWR032" H 1250 7150 50  0001 C CNN
+F 1 "Earth" H 1250 7250 50  0001 C CNN
+F 2 "" H 1250 7400 50  0001 C CNN
+F 3 "" H 1250 7400 50  0001 C CNN
+	1    1250 7400
+	0    -1   -1   0
+$EndComp
