File: Schamatic/Sensor-Infineon/Sensor.kicad_pcb (KiCad board)
At the start: 2 copper layers, 13.2 x 9.1 mm, 3 parts, among them J1 CONN_01X06, U1 TLE5012B

Commit message: new board version ready to order
Parts:
- J1: footprint Dizzy:SPI_cable -> Dizzy:SPI_CONN
- moved C1 9.59 mm to (-4.76, -0.02), turned to 90 degrees
- moved J1 4.66 mm to (0.14, 0.68)
- turned U1 to 180 degrees
Connections:
- J1 pad 1: MOSI -> +3V3
- J1 pad 2: MISO -> Earth
- J1 pad 3: CSK -> CS
- J1 pad 4: CS -> CSK
- J1 pad 5: Earth -> MISO
- J1 pad 6: +3V3 -> MOSI
Routing:
- net MOSI: track 6.33 -> 3.28 mm
- net MISO: track 2.12 -> 0.00 mm
- net +3V3: track 7.00 -> 4.99 mm
- net Earth: track 5.59 -> 6.41 mm
