File: Schamatic/Sensor-Infineon/Sensor.sch (KiCad schematic (older format))
At the start: 3 parts, among them J1 CONN_01X06, U1 TLE5012B

Commit message: new board version ready to order
Parts:
- J1: footprint Dizzy:SPI_cable -> Dizzy:SPI_CONN
Connections:
- net +3V3: now also J1.1 (P1); no longer J1.6 (P6)
- net CS: now also J1.3 (P3); no longer J1.4 (P4)
- net CSK: now also J1.4 (P4); no longer J1.3 (P3)
- net Earth: now also J1.2 (P2); no longer J1.5 (P5)
- net MISO: now also J1.5 (P5); no longer J1.2 (P2)
- net MOSI: now also J1.6 (P6); no longer J1.1 (P1)
Changed lines of the file:
@@
 LIBS:valves
 LIBS:Dizzy
+LIBS:Sensor-cache
 EELAYER 25 0
 EELAYER END
@@
 F 0 "J1" H 3550 3750 50  0000 C CNN
 F 1 "CONN_01X06" V 3650 3400 50  0000 C CNN
-F 2 "Dizzy:SPI_cable" H 3550 3400 50  0001 C CNN
+F 2 "Dizzy:SPI_CONN" H 3550 3400 50  0001 C CNN
 F 3 "" H 3550 3400 50  0001 C CNN
 	1    3550 3400
@@
 $EndComp
 $Comp
-L +3.3V #PWR1
+L +3.3V #PWR01
 U 1 1 59CE2D09
-P 3750 3150
-F 0 "#PWR1" H 3750 3000 50  0001 C CNN
-F 1 "+3.3V" H 3750 3290 50  0000 C CNN
-F 2 "" H 3750 3150 50  0001 C CNN
-F 3 "" H 3750 3150 50  0001 C CNN
-	1    3750 3150
+P 3750 3650
+F 0 "#PWR01" H 3750 3500 50  0001 C CNN
+F 1 "+3.3V" H 3750 3790 50  0000 C CNN
+F 2 "" H 3750 3650 50  0001 C CNN
+F 3 "" H 3750 3650 50  0001 C CNN
+	1    3750 3650
 	0    1    1    0
 $EndComp
 $Comp
-L Earth #PWR2
+L Earth #PWR02
 U 1 1 59CE2D23
-P 3750 3250
-F 0 "#PWR2" H 3750 3000 50  0001 C CNN
-F 1 "Earth" H 3750 3100 50  0001 C CNN
-F 2 "" H 3750 3250 50  0001 C CNN
-F 3 "" H 3750 3250 50  0001 C CNN
-	1    3750 3250
+P 3750 3550
+F 0 "#PWR02" H 3750 3300 50  0001 C CNN
+F 1 "Earth" H 3750 3400 50  0001 C CNN
+F 2 "" H 3750 3550 50  0001 C CNN
+F 3 "" H 3750 3550 50  0001 C CNN
+	1    3750 3550
 	0    -1   -1   0
 $EndComp
+Text GLabel 3750 3450 2    60   Input ~ 0
+CS
 Text GLabel 3750 3350 2    60   Input ~ 0
-CS
-Text GLabel 3750 3450 2    60   Input ~ 0
 CSK
-Text GLabel 3750 3550 2    60   Input ~ 0
+Text GLabel 3750 3250 2    60   Input ~ 0
 MISO
-Text GLabel 3750 3650 2    60   Input ~ 0
+Text GLabel 3750 3150 2    60   Input ~ 0
 MOSI
 $Comp
-L Earth #PWR3
+L Earth #PWR03
 U 1 1 59CE2D8E
 P 5850 3350
-F 0 "#PWR3" H 5850 3100 50  0001 C CNN
+F 0 "#PWR03" H 5850 3100 50  0001 C CNN
 F 1 "Earth" H 5850 3200 50  0001 C CNN
 F 2 "" H 5850 3350 50  0001 C CNN
@@
 $EndComp
 $Comp
-L +3.3V #PWR4
+L +3.3V #PWR04
 U 1 1 59CE2DA2
 P 5900 3500
-F 0 "#PWR4" H 5900 3350 50  0001 C CNN
+F 0 "#PWR04" H 5900 3350 50  0001 C CNN
 F 1 "+3.3V" H 5900 3640 50  0000 C CNN
 F 2 "" H 5900 3500 50  0001 C CNN
