File: Schamatic/Mainboard/Mainboard.sch (KiCad schematic (older format))
At the start: 7 parts

Commit message: continue mainboard
Parts:
- removed J?: CONN_02X20, symbol CONN_02X20
- added C? (x2): GRM31CR60J226KE19, symbol C_Small
- added C?: C_Small, symbol C_Small
- added C? (x15): 0.1uF, symbol C_Small
- added C? (x2): 10uF, symbol C_Small
- added C? (x2): 22uF, symbol C_Small
- added C?: 1uF, symbol C_Small
- added D?: SSA33L, symbol D
- added D?: D, symbol D
- added J?: BAT, symbol CONN_01X02
- added J?: JTAG, symbol CONN_01X05
- added L?: VLF10040T-6R8N4R5, symbol L
- added L?: 1uH, symbol L
- added L? (x2): 2.2uH, symbol L
- added L?: 10uH, symbol L
- added Q?: BSC030P03NS3GAUMA1, symbol Q_PMOS_DGS
- added R? (x3): 100k, symbol R
- added R?: R, symbol R
- added SW?: B3U-1000P, symbol B3U-1000P
- added U?: cc3220, symbol cc3220
- added U?: MX25R3235F, symbol MX25R3235F
- U?: value ADP2303ARDZ-5.0-R7 -> ADP2303ARDZ-3.3
Connections:
- net labels added: 12V, 3v3, ANA_SW, DIG_SW, Earth, JTAG_TCK, JTAG_TDI, JTAG_TDO, JTAG_TMS, SFL_CLK, SFL_CS, SFL_DIN, SFL_DOUT, VDD_ANA, VDD_DIG, VDD_PA
- net labels removed: +3.3V, +5V, MISO, MOSI, SCK
- wire segments 36 -> 88
- no-connect marks 0 -> 3
Other:
- moved on the sheet: C?, U?

Commit message: working on mainboard PCB
Parts:
- removed J?: JTAG, symbol CONN_01X05
- added AE1: AH316M245001-T, symbol Antenna_Dipole
- added C23, C29: 6.2pF, symbol C_Small
- added C24, C28, C3, C4: C_Small, symbol C_Small
- added C26: 0.5pF, symbol C_Small
- added D2, D4, D5, D6, D7: LED, symbol LED
- added J2: MOTORS, symbol CONN_01X02
- added J3: USART, symbol CONN_01X02
- added J4: 3.3V, symbol CONN_01X02
- added J5: CONN_01X07, symbol CONN_01X07
- added J6: FTSH-105-01-F-D-K, symbol CONN_02X05
- added L6: 3.3nh, symbol L
- added R1: 1k, symbol R
- added R10, R11, R12, R9: 300, symbol R
- added R14, R15: 3k, symbol R
- added R4, R5, R7, R8: R, symbol R
- added R6: 1.2k, symbol R
- added SW2, SW3, SW4: B3U-1000P, symbol B3U-1000P
- added U1: ACS781, symbol ACS781
- added U4: DEA202450BT, symbol DEA202450BT
- added Y1: Crystal, symbol Crystal
- added Y2: 40MHz, symbol Crystal_GND23
- C13: renamed from C?; value 0.1uF -> 10uF
- C31, C32: renamed from C?; value 100n -> 0.1uF
- C33: renamed from C?; value 47u -> 47uF
- C34: renamed from C?; value 10n -> 10n 16V
- gave numbers to parts that had none: 40
Connections:
- net labels added: ADC_I, ADC_V, GPIO14, GPIO15, GPIO16, GPIO17, GPIO18, RTC_N, RTC_P, RX, TX, XTAL_N, XTAL_P, nRESET
- net labels removed: GND
- wire segments 88 -> 117
- no-connect marks 3 -> 19
Other:
- moved on the sheet: D1, J1, Q1, R2, SW1

Commit message: started assigning footprints for motherboard
Parts:
- removed J5: CONN_01X07, symbol CONN_01X07
- added J5: CONN_02X04, symbol CONN_02X04
- C1: value C_Small -> 22uF; footprint (none) -> Capacitors_SMD:C_0805
- C10, C11, C13, C21, C25, C27, C33: footprint (none) -> Capacitors_SMD:C_0805
- C12, C14, C15, C16, C17, C18, C19, C20, C22, C23, C26, C29, C30, C31, C32, C34, C7, C8, C9: footprint (none) -> Capacitors_SMD:C_0603
- C2: value 0.1uF -> 0.1uF 25V; footprint (none) -> Capacitors_SMD:C_0603
- C24, C28: value C_Small -> 10pF; footprint (none) -> Capacitors_SMD:C_0603
- C3, C4: value C_Small -> 0.01uF; footprint (none) -> Capacitors_SMD:C_0603
- C5, C6: footprint (none) -> Capacitors_SMD:C_1206
- D2, D3: footprint (none) -> Diodes_SMD:D_SMA
- D4, D5, D6, D7: footprint (none) -> LEDs:LED_0603
- R1, R10, R11, R12, R13, R14, R15, R16, R2, R3, R4, R5, R6, R7, R8, R9: footprint (none) -> Resistors_SMD:R_0603
- U1: footprint (none) -> Dizzy:ACS781
- U2: footprint (none) -> Housings_SOIC:HTSOP-8-1EP_3.9x4.9mm_Pitch1.27mm
- U3: footprint (none) -> Housings_QFP:TQFP-64-1EP_10x10mm_Pitch0.5mm
- Y1: value Crystal -> 32.768kHz
- Y2: footprint (none) -> Dizzy:Crystal-250X200X55N
Connections:
- net labels added: GPIO0, GPIO4, GPIO5, GPIO6, GPIO7, GPIO8
- net labels removed: GPIO14, GPIO15, GPIO16, GPIO17, GPIO18
- no-connect marks 19 -> 18

Commit message: assigned all footprints for motherboard
Parts:
- removed D1: D, symbol D
- removed J1: BAT, symbol CONN_01X02
- removed J2: MOTORS, symbol CONN_01X02
- removed L4: 10uH, symbol L
- added J1: BAT+, Connectors:1pin, symbol CONN_01X01
- added J10: BAT-, Connectors:1pin, symbol CONN_01X01
- added J2: M+1, Connectors:1pin, symbol CONN_01X01
- added J7: M+2, Connectors:1pin, symbol CONN_01X01
- added J8: M-1, Connectors:1pin, symbol CONN_01X01
- added J9: M-2, Connectors:1pin, symbol CONN_01X01
- AE1: footprint (none) -> Dizzy:AH316M
- D2: footprint Diodes_SMD:D_SMA -> LEDs:LED_0603
- J3, J4: footprint (none) -> Pin_Headers:Pin_Header_Straight_2x01_Pitch2.54mm
- J5: footprint (none) -> Pin_Headers:Pin_Header_Straight_2x04_Pitch2.54mm
- J6: footprint (none) -> Pin_Headers:Pin_Header_Straight_2x05_Pitch1.27mm
- L1: footprint (none) -> Dizzy:VLF10040
- L2, L3, L5: footprint (none) -> Inductors_NEOSID:Neosid_Inductor_SM-NE29_SMD1008
- L6: footprint (none) -> Inductors_SMD:L_0603
- Q1: footprint (none) -> Dizzy:BSC030P
- SW1, SW2, SW3, SW4: footprint (none) -> Resistors_SMD:R_1206
- U4: footprint (none) -> Dizzy:DEA202450BT
- U5: footprint (none) -> Housings_SOIC:SOIJ-8_5.3x5.3mm_Pitch1.27mm
- U6: footprint (none) -> Housings_LGA:LGA-24L_3x3.5mm_Pitch0.43mm
- Y1: footprint (none) -> Crystals:Crystal_SMD_MicroCrystal_CC7V-T1A-2pin_3.2x1.5mm
- Y2: value 40MHz -> 40Mhz
Connections:
- net 12V: now also Q1.1 (D), R4.1, U1.5 (I+)
- net Earth: now also J10.1 (P1), J8.1 (P1), J9.1 (P1)
- net at Q1.3 (S), R2.2: now also J1.1 (P1)
- net at U1.6 (I-): now also J2.1 (P1), J7.1 (P1)
- no-connect marks 18 -> 20

Commit message: pushbutton switch
Parts:
- added C?: 0.1uF, symbol C_Small
- added R? (x2): 100k, symbol R
- added R?: 1.4M, symbol R
- added U?: LTC2954, symbol LTC2954
- R2: value R -> 100k
Connections:
- net Earth: now also SW1.1, C?.1, R?.1, U?.1 (GND), U?.9 (PAD); no longer SW1.2
- net at J1.1 (P1), Q1.3 (S), R2.2: now also C?.2, U?.4 (VIN)
- new net: Q1.2 (G), R?.2
- new net: R2.1, R?.1, R?.2, U?.7 (~EN)
- new net: SW1.2, U?.3 (~PB)
- new net: R?.1, R?.2, U?.5 (~KILL)
- no-connect marks 20 -> 23
Other:
- moved on the sheet: C1, C2, C3, C4, C5, C6, D2, D3, D4, J1, J10, J2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

Commit message: continue motherboard
Parts:
- added C36: 0.1uF, Capacitors_SMD:C_0603, symbol C_Small
- added D1, D8: D, Diodes_SMD:D_SMA, symbol D
- added J11: PLUG+, Connectors:1pin, symbol CONN_01X01
- added J12: PLUG-, Connectors:1pin, symbol CONN_01X01
- added U8: LTC2876, Dizzy:LTC2876, symbol LTC2876
- C35: renamed from C?; footprint (none) -> Capacitors_SMD:C_0603
- Q1: value BSC030P03NS3GAUMA1 -> p-MOSFET
- R17, R18, R19: renamed from R?; footprint (none) -> Resistors_SMD:R_0603
- U7: renamed from U?; footprint (none) -> Housings_DFN_QFN:DFN-8-1EP_2x3mm_Pitch0.5mm
Connections:
- net 3v3: now also C36.2, U8.8 (VCC)
- net Earth: now also C36.1, J12.1 (P1), U8.2 (~RE), U8.5 (GND), U8.9 (PAD)
- net RX: now also U8.1 (RO); no longer J3.1 (P1)
- net TX: now also U8.4 (DI); no longer J3.2 (P2)
- net DE: now reaches U3.3 (GPIO12)
- net DE: now also U8.3 (DE)
- net at C35.2, Q1.3 (S), R2.2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: now also D1.1 (K), D8.1 (K); no longer J1.1 (P1)
- new net: D8.2 (A), J1.1 (P1)
- new net: D1.2 (A), J11.1 (P1)
- new net RS-A: J3.2 (P2), U8.7 (A)
- new net RS-B: J3.1 (P1), U8.6 (B)
Other:
- moved on the sheet: C3, C35, C4, D2, J1, J10, J2, J7, J8, J9, Q1, R17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

Commit message: working on mainboard PCB
Parts:
- added J13, J14, J15, J16: MOUNT, Mounting_Holes:MountingHole_3.5mm_Pad, symbol CONN_01X01
- added SW5: B3U-1000P, Resistors_SMD:R_1206, symbol B3U-1000P
- AE1: value AH316M245001-T -> ANT
Connections:
- net 3v3: now also SW5.1
- net Earth: now also J13.1 (P1), J14.1 (P1), J15.1 (P1), J16.1 (P1)
- net at U3.53 (GPIO30): now also SW5.2
- no-connect marks 23 -> 21
Changed lines of the file:
@@
 P 12050 3550
 F 0 "AE1" H 12100 3600 50  0000 C CNN
-F 1 "AH316M245001-T" H 12100 3550 50  0000 C CNN
+F 1 "ANT" H 12100 3550 50  0000 C CNN
 F 2 "Dizzy:AH316M" H 12050 3550 50  0001 C CNN
-F 3 "" H 12050 3550 50  0001 C CNN
+F 3 "AH316M245001-T" H 12050 3550 50  0001 C CNN
 	1    12050 3550
 	1    0    0    -1
@@
 	0    1    1    0
 $EndComp
-NoConn ~ 6350 4250
 NoConn ~ 6350 4550
-NoConn ~ 6950 6200
 Wire Wire Line
 	12850 1500 13250 1500
@@
 Wire Wire Line
 	1600 9300 1350 9300
+$Comp
+L B3U-1000P SW5
+U 1 1 5A50A0FE
+P 6100 4800
+F 0 "SW5" H 6050 5100 60  0000 C CNN
+F 1 "B3U-1000P" H 6100 5250 60  0000 C CNN
+F 2 "Resistors_SMD:R_1206" H 6100 4800 60  0001 C CNN
+F 3 "" H 6100 4800 60  0001 C CNN
+	1    6100 4800
+	1    0    0    -1
+$EndComp
+Text GLabel 5800 4250 0    60   Input ~ 0
+3v3
+$Comp
+L CONN_01X01 J13
+U 1 1 5A51026A
+P 950 2150
+F 0 "J13" H 950 2250 50  0000 C CNN
+F 1 "MOUNT" H 1150 2150 50  0000 C CNN
+F 2 "Mounting_Holes:MountingHole_3.5mm_Pad" H 950 2150 50  0001 C CNN
+F 3 "" H 950 2150 50  0001 C CNN
+	1    950  2150
+	-1   0    0    1
+$EndComp
+$Comp
+L CONN_01X01 J14
+U 1 1 5A51038B
+P 950 2350
+F 0 "J14" H 950 2450 50  0000 C CNN
+F 1 "MOUNT" H 1150 2350 50  0000 C CNN
+F 2 "Mounting_Holes:MountingHole_3.5mm_Pad" H 950 2350 50  0001 C CNN
+F 3 "" H 950 2350 50  0001 C CNN
+	1    950  2350
+	-1   0    0    1
+$EndComp
+$Comp
+L CONN_01X01 J16
+U 1 1 5A51047E
+P 950 2750
+F 0 "J16" H 950 2850 50  0000 C CNN
+F 1 "MOUNT" H 1150 2750 50  0000 C CNN
+F 2 "Mounting_Holes:MountingHole_3.5mm_Pad" H 950 2750 50  0001 C CNN
+F 3 "" H 950 2750 50  0001 C CNN
+	1    950  2750
+	-1   0    0    1
+$EndComp
+$Comp
+L CONN_01X01 J15
+U 1 1 5A51055B
+P 950 2550
+F 0 "J15" H 950 2650 50  0000 C CNN
+F 1 "MOUNT" H 1150 2550 50  0000 C CNN
+F 2 "Mounting_Holes:MountingHole_3.5mm_Pad" H 950 2550 50  0001 C CNN
+F 3 "" H 950 2550 50  0001 C CNN
+	1    950  2550
+	-1   0    0    1
+$EndComp
+$Comp
+L Earth #PWR072
+U 1 1 5A512606
+P 1150 2750
+F 0 "#PWR072" H 1150 2500 50  0001 C CNN
+F 1 "Earth" H 1150 2600 50  0001 C CNN
+F 2 "" H 1150 2750 50  0001 C CNN
+F 3 "" H 1150 2750 50  0001 C CNN
+	1    1150 2750
+	0    -1   -1   0
+$EndComp
+$Comp
+L Earth #PWR073
+U 1 1 5A51389C
+P 1150 2550
+F 0 "#PWR073" H 1150 2300 50  0001 C CNN
+F 1 "Earth" H 1150 2400 50  0001 C CNN
+F 2 "" H 1150 2550 50  0001 C CNN
+F 3 "" H 1150 2550 50  0001 C CNN
+	1    1150 2550
+	0    -1   -1   0
+$EndComp
+$Comp
+L Earth #PWR074
+U 1 1 5A5139D6
+P 1150 2350
+F 0 "#PWR074" H 1150 2100 50  0001 C CNN
+F 1 "Earth" H 1150 2200 50  0001 C CNN
+F 2 "" H 1150 2350 50  0001 C CNN
+F 3 "" H 1150 2350 50  0001 C CNN
+	1    1150 2350
+	0    -1   -1   0
+$EndComp
+$Comp
+L Earth #PWR075
+U 1 1 5A513B10
+P 1150 2150
+F 0 "#PWR075" H 1150 1900 50  0001 C CNN
+F 1 "Earth" H 1150 2000 50  0001 C CNN
+F 2 "" H 1150 2150 50  0001 C CNN
+F 3 "" H 1150 2150 50  0001 C CNN
+	1    1150 2150
+	0    -1   -1   0
+$EndComp
 $EndSCHEMATC

Commit message: motherboard minor changes
Parts:
- removed U4: DEA202450BT, Dizzy:DEA202450BT, symbol DEA202450BT
- added U4: DEA202450BT-3201B2, Dizzy:DEA202450BT-3201B2, symbol DEA202450BT-3201B2
- C3, C4: value 0.01uF -> 0.1uF 25V
- J6: value FTSH-105-01-F-D-K -> JTAG
- R18: value 1.4M -> 140K
- R19: value 100k -> 10k
- R4: value R -> 200K 1%
- R5: value R -> 10K 1%
- R7: value R -> 22k 1%
- R8: value R -> 10k 1%
Connections:
- net Earth: now also U4.1 (GND), U4.3 (GND), U4.4 (GND), U4.6 (GND)
- net at U3.31 (RF_BG): now also U4.2 (IN)
- net at L6.1: now also U4.5 (OUT)
Other:
- moved on the sheet: AE1, C26, L6
