File: Schamatic/Mainboard/Mainboard.sch (KiCad schematic (older format))
At the start: 101 parts, among them J1 BAT+, J10 BAT-, J11 PLUG+, J12 PLUG-, J13 MOUNT, J14 MOUNT, J15 MOUNT, J16 MOUNT, J2 M+1, J3 USART, J4 3.3V, J5 CONN_02X04, J6 JTAG, J7 M+2, J8 M-1, J9 M-2, Q1 p-MOSFET, SW1 B3U-1000P, SW2 B3U-1000P, SW3 B3U-1000P, SW4 B3U-1000P, SW5 B3U-1000P, U1 ACS781, U2 ADP2303ARDZ-3.3, U3 cc3220, U4 DEA202450BT-3201B2, U5 MX25R3235F, U6 LSM9DS1, U7 LTC2954, U8 LTC2876, Y1 32.768kHz, Y2 40Mhz

Commit message: whatever motherboard changes
Parts:
- U3: footprint Housings_QFP:TQFP-64-1EP_10x10mm_Pitch0.5mm -> Housings_DFN_QFN:QFN-64-1EP_9x9mm_Pitch0.5mm
Connections:
- net 3v3: now also J5.7 (P7); no longer J5.2 (P2)
- net ADC_V: now also U3.59 (GPIO4); no longer U3.57 (GPIO2)
- net GPIO6: now also J5.5 (P5); no longer J5.6 (P6)
- net GPIO7: now also J5.6 (P6); no longer J5.7 (P7)
- net nRESET: now also J5.3 (P3)
- net FLASH_TX: now reaches U3.55 (GPIO1)
- net FLASH_TX: now also J5.2 (P2)
- net GPIO0: no longer names the net of U3.50 (GPIO0)
- net GPIO0: no longer J5.3 (P3)
- net GPIO4 renamed FLASH_RX
- net FLASH_RX: now also U3.57 (GPIO2); no longer U3.59 (GPIO4)
- net GPIO5: no longer names the net of U3.60 (GPIO5)
- net GPIO5: no longer J5.5 (P5)
- no-connect marks 21 -> 20

Commit message: minor corrections
Parts:
- C3, C4: value 0.1uF 25V -> 0.1uF
- C5, C6: value GRM31CR60J226KE19 -> 22uF
Changed lines of the file:
@@
 P 9050 9850
 F 0 "C5" H 9060 9920 50  0000 L CNN
-F 1 "GRM31CR60J226KE19" H 9060 9770 50  0000 L CNN
+F 1 "22uF" H 9060 9770 50  0000 L CNN
 F 2 "Capacitors_SMD:C_1206" H 9050 9850 50  0001 C CNN
 F 3 "" H 9050 9850 50  0001 C CNN
@@
 P 9350 9850
 F 0 "C6" H 9360 9920 50  0000 L CNN
-F 1 "GRM31CR60J226KE19" H 9360 9770 50  0000 L CNN
+F 1 "22uF" H 9360 9770 50  0000 L CNN
 F 2 "Capacitors_SMD:C_1206" H 9350 9850 50  0001 C CNN
 F 3 "" H 9350 9850 50  0001 C CNN
@@
 P 2900 9100
 F 0 "C3" H 2910 9170 50  0000 L CNN
-F 1 "0.1uF 25V" H 2910 9020 50  0000 L CNN
+F 1 "0.1uF" H 2910 9020 50  0000 L CNN
 F 2 "Capacitors_SMD:C_0603" H 2900 9100 50  0001 C CNN
 F 3 "" H 2900 9100 50  0001 C CNN
@@
 P 3800 9500
 F 0 "C4" H 3810 9570 50  0000 L CNN
-F 1 "0.1uF 25V" H 3810 9420 50  0000 L CNN
+F 1 "0.1uF" H 3810 9420 50  0000 L CNN
 F 2 "Capacitors_SMD:C_0603" H 3800 9500 50  0001 C CNN
 F 3 "" H 3800 9500 50  0001 C CNN

Commit message: SolidWorks 3D
Connections:
- net at C35.2, D1.1 (K), D8.1 (K)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: now also R18.2
- net at R17.1, R2.1, U7.7 (~EN): no longer R18.2
Other:
- moved on the sheet: C35, R18, R19, SW1
Changed lines of the file:
@@
 L B3U-1000P SW1
 U 1 1 5A43A034
-P 1750 7250
-F 0 "SW1" H 1700 7550 60  0000 C CNN
-F 1 "B3U-1000P" H 1750 7700 60  0000 C CNN
-F 2 "Resistors_SMD:R_1206" H 1750 7250 60  0001 C CNN
-F 3 "" H 1750 7250 60  0001 C CNN
-	1    1750 7250
+P 1450 7250
+F 0 "SW1" H 1400 7550 60  0000 C CNN
+F 1 "B3U-1000P" H 1450 7700 60  0000 C CNN
+F 2 "Resistors_SMD:R_1206" H 1450 7250 60  0001 C CNN
+F 3 "" H 1450 7250 60  0001 C CNN
+	1    1450 7250
 	0    -1   -1   0
 $EndComp
@@
 L Earth #PWR08
 U 1 1 5A43A0C3
-P 1200 7550
-F 0 "#PWR08" H 1200 7300 50  0001 C CNN
-F 1 "Earth" H 1200 7400 50  0001 C CNN
-F 2 "" H 1200 7550 50  0001 C CNN
-F 3 "" H 1200 7550 50  0001 C CNN
-	1    1200 7550
+P 900 7550
+F 0 "#PWR08" H 900 7300 50  0001 C CNN
+F 1 "Earth" H 900 7400 50  0001 C CNN
+F 2 "" H 900 7550 50  0001 C CNN
+F 3 "" H 900 7550 50  0001 C CNN
+	1    900  7550
 	1    0    0    -1
 $EndComp
@@
 $EndComp
 Wire Wire Line
-	1200 7000 1600 7000
+	900  7000 1600 7000
 Wire Wire Line
 	1600 7150 1600 9300
@@
 L R R18
 U 1 1 5A4BB197
-P 2850 7350
-F 0 "R18" V 2930 7350 50  0000 C CNN
-F 1 "140K" V 2850 7350 50  0000 C CNN
-F 2 "Resistors_SMD:R_0603" V 2780 7350 50  0001 C CNN
-F 3 "" H 2850 7350 50  0001 C CNN
-	1    2850 7350
-	0    1    1    0
+P 1450 7300
+F 0 "R18" V 1530 7300 50  0000 C CNN
+F 1 "140K" V 1450 7300 50  0000 C CNN
+F 2 "Resistors_SMD:R_0603" V 1380 7300 50  0001 C CNN
+F 3 "" H 1450 7300 50  0001 C CNN
+	1    1450 7300
+	-1   0    0    1
 $EndComp
 $Comp
 L R R19
 U 1 1 5A4BB290
-P 3150 7350
-F 0 "R19" V 3230 7350 50  0000 C CNN
-F 1 "10k" V 3150 7350 50  0000 C CNN
-F 2 "Resistors_SMD:R_0603" V 3080 7350 50  0001 C CNN
-F 3 "" H 3150 7350 50  0001 C CNN
-	1    3150 7350
-	0    1    1    0
+P 1450 7600
+F 0 "R19" V 1530 7600 50  0000 C CNN
+F 1 "10k" V 1450 7600 50  0000 C CNN
+F 2 "Resistors_SMD:R_0603" V 1380 7600 50  0001 C CNN
+F 3 "" H 1450 7600 50  0001 C CNN
+	1    1450 7600
+	-1   0    0    1
 $EndComp
 $Comp
 L Earth #PWR065
 U 1 1 5A4BB3C2
-P 3300 7350
-F 0 "#PWR065" H 3300 7100 50  0001 C CNN
-F 1 "Earth" H 3300 7200 50  0001 C CNN
-F 2 "" H 3300 7350 50  0001 C CNN
-F 3 "" H 3300 7350 50  0001 C CNN
-	1    3300 7350
-	0    -1   -1   0
+P 1450 7750
+F 0 "#PWR065" H 1450 7500 50  0001 C CNN
+F 1 "Earth" H 1450 7600 50  0001 C CNN
+F 2 "" H 1450 7750 50  0001 C CNN
+F 3 "" H 1450 7750 50  0001 C CNN
+	1    1450 7750
+	1    0    0    -1
 $EndComp
 Wire Wire Line
 	2500 7150 3000 7150
 Wire Wire Line
-	3000 7150 3000 7350
-Connection ~ 3000 7350
-Connection ~ 2700 7350
+	3000 7150 3000 7600
 Wire Wire Line
 	2700 7900 2700 6850
@@
 L C_Small C35
 U 1 1 5A4BBA39
-P 1450 7300
-F 0 "C35" H 1460 7370 50  0000 L CNN
-F 1 "0.1uF" H 1460 7220 50  0000 L CNN
-F 2 "Capacitors_SMD:C_0603" H 1450 7300 50  0001 C CNN
-F 3 "" H 1450 7300 50  0001 C CNN
-	1    1450 7300
-	-1   0    0    1
-$EndComp
-Wire Wire Line
-	1600 7150 1450 7150
-Wire Wire Line
-	1450 7150 1450 7200
+P 1150 7300
+F 0 "C35" H 1160 7370 50  0000 L CNN
+F 1 "0.1uF" H 1160 7220 50  0000 L CNN
+F 2 "Capacitors_SMD:C_0603" H 1150 7300 50  0001 C CNN
+F 3 "" H 1150 7300 50  0001 C CNN
+	1    1150 7300
+	-1   0    0    1
+$EndComp
+Wire Wire Line
+	1150 7150 1600 7150
+Wire Wire Line
+	1150 7150 1150 7200
 Connection ~ 1600 7150
 $Comp
 L Earth #PWR066
 U 1 1 5A4BBFDE
-P 1450 7550
-F 0 "#PWR066" H 1450 7300 50  0001 C CNN
-F 1 "Earth" H 1450 7400 50  0001 C CNN
-F 2 "" H 1450 7550 50  0001 C CNN
-F 3 "" H 1450 7550 50  0001 C CNN
-	1    1450 7550
-	1    0    0    -1
-$EndComp
-Wire Wire Line
-	1450 7400 1450 7550
+P 1150 7550
+F 0 "#PWR066" H 1150 7300 50  0001 C CNN
+F 1 "Earth" H 1150 7400 50  0001 C CNN
+F 2 "" H 1150 7550 50  0001 C CNN
+F 3 "" H 1150 7550 50  0001 C CNN
+	1    1150 7550
+	1    0    0    -1
+$EndComp
+Wire Wire Line
+	1150 7400 1150 7550
 $Comp
 L LTC2876 U8
@@
 Text GLabel 1250 5500 0    60   Input ~ 0
 GPIO6
+Connection ~ 1450 7150
+Wire Wire Line
+	1450 7450 1800 7450
+Wire Wire Line
+	1800 7450 1800 7600
+Wire Wire Line
+	1800 7600 3000 7600
+Connection ~ 1450 7450
 $EndSCHEMATC

Commit message: motherboard corrections
Parts:
- added R20: 100K, Resistors_SMD:R_0603, symbol R_Small
- added R21: 270, Resistors_SMD:R_0603, symbol R_Small
- added R22: 2.7K, Resistors_SMD:R_0603, symbol R_Small
- C27: footprint Capacitors_SMD:C_0805 -> Capacitors_SMD:C_0603
- R10, R11, R12, R9: value 300 -> 470
- R6: value 1.2k -> 2k
Connections:
- net 3v3: now also R21.1
- net Earth: now also R20.1, R22.1
- net at U3.21 (SOP2): now also R22.2
- net at U3.34 (SOP1): now also R21.2
- net at U3.35 (SOP0): now also R20.2
- no-connect marks 20 -> 17

Commit message: BAU
Parts:
- C1: value 22uF -> 22uF 25V
- C35: value 0.1uF -> 0.1uF 25V
Changed lines of the file:
@@
 U 1 1 5A43873A
 P 6750 10050
-F 0 "C1" H 6760 10120 50  0000 L CNN
-F 1 "22uF" H 6760 9970 50  0000 L CNN
+F 0 "C1" H 6700 10100 50  0000 L CNN
+F 1 "22uF 25V" H 6550 9950 50  0000 L CNN
 F 2 "Capacitors_SMD:C_0805" H 6750 10050 50  0001 C CNN
 F 3 "" H 6750 10050 50  0001 C CNN
@@
 U 1 1 5A43A034
 P 1450 7250
-F 0 "SW1" H 1400 7550 60  0000 C CNN
-F 1 "B3U-1000P" H 1450 7700 60  0000 C CNN
+F 0 "SW1" H 1450 7900 60  0000 C CNN
+F 1 "B3U-1000P" H 1450 8000 60  0000 C CNN
 F 2 "Resistors_SMD:R_1206" H 1450 7250 60  0001 C CNN
 F 3 "" H 1450 7250 60  0001 C CNN
@@
 U 1 1 5A4BBA39
 P 1150 7300
-F 0 "C35" H 1160 7370 50  0000 L CNN
-F 1 "0.1uF" H 1160 7220 50  0000 L CNN
+F 0 "C35" H 1100 7400 50  0000 L CNN
+F 1 "0.1uF 25V" H 1100 7200 50  0000 L CNN
 F 2 "Capacitors_SMD:C_0603" H 1150 7300 50  0001 C CNN
 F 3 "" H 1150 7300 50  0001 C CNN
