File: Schamatic/Mainboard/Mainboard.kicad_pcb (KiCad board)
At the start: 4 copper layers, 60.3 x 55.7 mm, 288 parts, among them J1 BAT+, J10 BAT-, J11 PLUG+, J12 PLUG-, J13 MOUNT, J14 MOUNT, J15 MOUNT, J16 MOUNT, J2 M+1, J3 USART, J4 3.3V, J5 CONN_02X04, J6 JTAG, J7 M+2, J8 M-1, J9 M-2, Q1 p-MOSFET, SW1 B3U-1000P, SW2 B3U-1000P, SW3 B3U-1000P, SW4 B3U-1000P, SW5 B3U-1000P, U1 ACS781, U2 ADP2303ARDZ-3.3, U3 cc3220, U4 DEA202450BT-3201B2, U5 MX25R3235F, U6 LSM9DS1, U7 LTC2954, U8 LTC2876, Y1 32.768kHz, Y2 40Mhz

Commit message: whatever motherboard changes
Parts:
- removed the REF** at (105.8, 104.6)
- removed the REF** at (101.0, 117.6)
- removed the REF** at (125.4, 114.0)
- removed the REF** at (125.4, 114.8)
- removed the REF** at (125.4, 113.2)
- removed the REF** at (125.4, 107.6)
- removed the REF** at (125.4, 110.0)
- removed the REF** at (125.4, 108.4)
- removed the REF** at (125.4, 110.8)
- removed the REF** at (125.4, 109.2)
- removed the REF** at (124.6, 111.6)
- removed the REF** at (124.6, 112.4)
- removed the REF** at (92.3, 116.8)
- removed the REF** at (124.6, 114.0)
- removed the REF** at (124.6, 114.8)
- removed the REF** at (124.6, 113.2)
- removed the REF** at (124.6, 107.6)
- removed the REF** at (124.6, 110.0)
- removed the REF** at (124.6, 108.4)
- removed the REF** at (124.6, 110.8)
- removed the REF** at (124.6, 109.2)
- removed the REF** at (123.8, 111.6)
- removed the REF** at (123.8, 112.4)
- removed the REF** at (95.5, 123.2)
- removed the REF** at (123.8, 114.0)
- removed the REF** at (123.8, 114.8)
- removed the REF** at (123.8, 113.2)
- removed the REF** at (123.8, 107.6)
- removed the REF** at (123.8, 110.0)
- removed the REF** at (123.8, 108.4)
- removed the REF** at (123.8, 110.8)
- removed the REF** at (123.8, 109.2)
- removed the REF** at (123.0, 111.6)
- removed the REF** at (123.0, 112.4)
- removed the REF** at (118.8, 129.0)
- removed the REF** at (123.0, 114.0)
- removed the REF** at (123.0, 114.8)
- removed the REF** at (123.0, 113.2)
- removed the REF** at (123.0, 107.6)
- removed the REF** at (123.0, 110.0)
- removed the REF** at (123.0, 108.4)
- removed the REF** at (123.0, 110.8)
- removed the REF** at (123.0, 109.2)
- removed the REF** at (122.2, 111.6)
- removed the REF** at (122.2, 112.4)
- removed the REF** at (110.7, 129.0)
- removed the REF** at (122.2, 114.0)
- removed the REF** at (122.2, 114.8)
- removed the REF** at (122.2, 113.2)
- removed the REF** at (122.2, 107.6)
- removed the REF** at (122.2, 110.0)
- removed the REF** at (122.2, 108.4)
- removed the REF** at (122.2, 110.8)
- removed the REF** at (122.2, 109.2)
- removed the REF** at (121.4, 111.6)
- removed the REF** at (121.4, 112.4)
- removed the REF** at (114.1, 124.0)
- removed the REF** at (121.4, 114.0)
- removed the REF** at (121.4, 114.8)
- removed the REF** at (121.4, 113.2)
- removed the REF** at (121.4, 107.6)
- removed the REF** at (121.4, 110.0)
- removed the REF** at (121.4, 108.4)
- removed the REF** at (121.4, 110.8)
- removed the REF** at (121.4, 109.2)
- removed the REF** at (120.6, 111.6)
- removed the REF** at (120.6, 112.4)
- removed the REF** at (130.0, 126.2)
- removed the REF** at (120.6, 114.0)
- removed the REF** at (120.6, 114.8)
- removed the REF** at (120.6, 113.2)
- removed the REF** at (120.6, 107.6)
- removed the REF** at (120.6, 110.0)
- removed the REF** at (120.6, 108.4)
- removed the REF** at (120.6, 110.8)
- removed the REF** at (120.6, 109.2)
- removed the REF** at (119.8, 111.6)
- removed the REF** at (119.8, 112.4)
- removed the REF** at (129.3, 126.0)
- removed the REF** at (119.8, 114.0)
- removed the REF** at (119.8, 114.8)
- removed the REF** at (119.8, 113.2)
- removed the REF** at (119.8, 107.6)
- removed the REF** at (119.8, 110.0)
- removed the REF** at (119.8, 108.4)
- removed the REF** at (119.8, 110.8)
- removed the REF** at (119.8, 109.2)
- removed the REF** at (119.0, 114.8)
- removed the REF** at (119.0, 107.6)
- removed the REF** at (131.4, 127.2)
- removed the REF** at (119.0, 108.4)
- removed the REF** at (119.0, 109.2)
- removed the REF** at (119.0, 110.0)
- removed the REF** at (119.0, 110.8)
- removed the REF** at (119.0, 111.6)
- removed the REF** at (119.0, 112.4)
- removed the REF** at (119.0, 113.2)
- removed the REF** at (119.0, 114.0)
- removed the REF** at (129.4, 126.8)
- removed the REF** at (103.3, 112.2)
- removed the REF** at (128.5, 126.8)
- removed the REF** at (128.6, 125.2)
- removed the REF** at (128.6, 124.4)
- removed the REF** at (128.6, 126.0)
- removed the REF** at (128.6, 123.6)
- removed the REF** at (123.4, 129.0)
- removed the REF** at (123.4, 129.8)
- removed the REF** at (123.4, 131.4)
- removed the REF** at (123.4, 130.6)
- removed the REF** at (123.4, 127.4)
- removed the REF** at (106.4, 113.4)
- removed the REF** at (123.4, 128.2)
- removed the REF** at (124.0, 123.4)
- removed the REF** at (124.0, 120.2)
- removed the REF** at (124.0, 119.4)
- removed the REF** at (124.0, 121.0)
- removed the REF** at (124.0, 122.6)
- removed the REF** at (124.0, 121.8)
- removed the REF** at (127.8, 118.0)
- removed the REF** at (127.8, 118.8)
- removed the REF** at (127.8, 119.6)
- removed the REF** at (94.7, 105.8)
- removed the REF** at (127.8, 121.2)
- removed the REF** at (127.8, 120.4)
- removed the REF** at (127.8, 122.0)
- removed the REF** at (127.8, 125.2)
- removed the REF** at (127.8, 123.6)
- removed the REF** at (127.8, 122.8)
- removed the REF** at (127.8, 124.4)
- removed the REF** at (124.6, 118.8)
- removed the REF** at (130.6, 126.8)
- removed the REF** at (130.6, 127.6)
- removed the REF** at (103.7, 94.6)
- removed the REF** at (130.6, 129.2)
- removed the REF** at (130.6, 130.0)
- removed the REF** at (130.6, 128.4)
- removed the REF** at (131.4, 128.0)
- removed the REF** at (131.4, 130.4)
- removed the REF** at (131.4, 128.8)
- removed the REF** at (131.4, 131.2)
- removed the REF** at (131.4, 129.6)
- removed the REF** at (124.0, 128.2)
- removed the REF** at (124.0, 129.0)
- removed the REF** at (108.8, 93.0)
- removed the REF** at (124.0, 130.6)
- removed the REF** at (124.0, 131.4)
- removed the REF** at (124.0, 129.8)
- removed the REF** at (124.0, 124.2)
- removed the REF** at (124.0, 126.6)
- removed the REF** at (124.0, 125.0)
- removed the REF** at (124.0, 127.4)
- removed the REF** at (124.0, 125.8)
- removed the REF** at (127.0, 122.0)
- removed the REF** at (127.0, 122.8)
- removed the REF** at (99.6, 93.6)
- removed the REF** at (127.0, 124.4)
- removed the REF** at (127.0, 125.2)
- removed the REF** at (127.0, 123.6)
- removed the REF** at (127.0, 118.0)
- removed the REF** at (126.7, 120.5)
- removed the REF** at (127.0, 118.8)
- removed the REF** at (127.0, 121.2)
- removed the REF** at (127.0, 119.6)
- removed the REF** at (124.6, 123.4)
- removed the REF** at (124.6, 124.2)
- removed the REF** at (99.7, 96.4)
- removed the REF** at (124.6, 125.8)
- removed the REF** at (124.6, 126.6)
- removed the REF** at (124.6, 125.0)
- removed the REF** at (124.6, 119.6)
- removed the REF** at (124.6, 121.8)
- removed the REF** at (124.6, 121.2)
- removed the REF** at (124.6, 122.6)
- removed the REF** at (124.8, 120.5)
- removed the REF** at (126.2, 111.6)
- removed the REF** at (126.2, 112.4)
- removed the REF** at (99.7, 101.2)
- removed the REF** at (126.2, 114.0)
- removed the REF** at (126.2, 114.8)
- removed the REF** at (126.2, 113.2)
- removed the REF** at (126.2, 107.6)
- removed the REF** at (126.2, 110.0)
- removed the REF** at (126.2, 108.4)
- removed the REF** at (126.2, 110.8)
- removed the REF** at (126.2, 109.2)
- removed the REF** at (125.4, 111.6)
- removed the REF** at (125.4, 112.4)
- added REF**: VIA-0.4, Dizzy:VIA-0.4, F.Cu at (119.3, 129.0)
- added REF**: VIA-0.4, Dizzy:VIA-0.4, F.Cu at (98.7, 101.1)
- added REF**: VIA-0.4, Dizzy:VIA-0.4, F.Cu at (123.3, 126.4)
- added REF**: VIA-0.4, Dizzy:VIA-0.4, F.Cu at (123.3, 129.6)
- added REF**: VIA-0.4, Dizzy:VIA-0.4, F.Cu at (123.3, 131.2)
- added REF**: VIA-0.4, Dizzy:VIA-0.4, F.Cu at (123.3, 128.0)
- added REF**: VIA-0.4, Dizzy:VIA-0.4, F.Cu at (123.3, 128.8)
- added REF**: VIA-0.4, Dizzy:VIA-0.4, F.Cu at (123.3, 130.4)
- added REF**: VIA-0.4, Dizzy:VIA-0.4, F.Cu at (131.2, 126.7)
- added REF**: VIA-0.4, Dizzy:VIA-0.4, F.Cu at (131.2, 127.7)
- added REF**: VIA-0.4, Dizzy:VIA-0.4, F.Cu at (131.2, 130.9)
- added REF**: VIA-0.4, Dizzy:VIA-0.4, F.Cu at (130.7, 129.7)
- added REF**: VIA-0.4, Dizzy:VIA-0.4, F.Cu at (91.1, 107.4)
- added REF**: VIA-0.4, Dizzy:VIA-0.4, F.Cu at (131.2, 129.3)
- added REF**: VIA-0.4, Dizzy:VIA-0.4, F.Cu at (131.2, 128.5)
- added REF**: VIA-0.4, Dizzy:VIA-0.4, F.Cu at (131.2, 130.1)
- added REF**: VIA-0.4, Dizzy:VIA-0.4, F.Cu at (130.7, 128.1)
- added REF**: VIA-0.4, Dizzy:VIA-0.4, F.Cu at (130.7, 127.3)
- added REF**: VIA-0.4, Dizzy:VIA-0.4, F.Cu at (130.7, 128.9)
- added REF**: VIA-0.4, Dizzy:VIA-0.4, F.Cu at (130.5, 126.6)
- added REF**: VIA-0.4, Dizzy:VIA-0.4, F.Cu at (130.1, 126.1)
- added REF**: VIA-0.4, Dizzy:VIA-0.4, F.Cu at (129.7, 126.6)
- added REF**: VIA-0.4, Dizzy:VIA-0.4, F.Cu at (129.3, 126.1)
- added REF**: VIA-0.4, Dizzy:VIA-0.4, F.Cu at (90.7, 117.0)
- added REF**: VIA-0.4, Dizzy:VIA-0.4, F.Cu at (128.9, 126.6)
- added REF**: VIA-0.4, Dizzy:VIA-0.4, F.Cu at (128.1, 126.6)
- added REF**: VIA-0.4, Dizzy:VIA-0.4, F.Cu at (128.5, 126.1)
- added REF**: VIA-0.4, Dizzy:VIA-0.4, F.Cu at (128.5, 125.2)
- added REF**: VIA-0.4, Dizzy:VIA-0.4, F.Cu at (128.1, 125.7)
- added REF**: VIA-0.4, Dizzy:VIA-0.4, F.Cu at (127.7, 125.2)
- added REF**: VIA-0.4, Dizzy:VIA-0.4, F.Cu at (124.3, 126.4)
- added REF**: VIA-0.4, Dizzy:VIA-0.4, F.Cu at (124.3, 125.6)
- added REF**: VIA-0.4, Dizzy:VIA-0.4, F.Cu at (124.8, 121.3)
- added REF**: VIA-0.4, Dizzy:VIA-0.4, F.Cu at (126.7, 121.3)
- added REF**: VIA-0.4, Dizzy:VIA-0.4, F.Cu at (98.4, 114.0)
- added REF**: VIA-0.4, Dizzy:VIA-0.4, F.Cu at (126.7, 118.1)
- added REF**: VIA-0.4, Dizzy:VIA-0.4, F.Cu at (126.7, 118.9)
- added REF**: VIA-0.4, Dizzy:VIA-0.4, F.Cu at (124.8, 118.0)
- added REF**: VIA-0.4, Dizzy:VIA-0.4, F.Cu at (124.8, 118.9)
- added REF**: VIA-0.4, Dizzy:VIA-0.4, F.Cu at (123.7, 118.1)
- added REF**: VIA-0.4, Dizzy:VIA-0.4, F.Cu at (123.7, 118.9)
- added REF**: VIA-0.4, Dizzy:VIA-0.4, F.Cu at (123.7, 120.4)
- added REF**: VIA-0.4, Dizzy:VIA-0.4, F.Cu at (123.7, 119.6)
- added REF**: VIA-0.4, Dizzy:VIA-0.4, F.Cu at (123.7, 121.2)
- added REF**: VIA-0.4, Dizzy:VIA-0.4, F.Cu at (123.8, 122.8)
- added REF**: VIA-0.4, Dizzy:VIA-0.4, F.Cu at (106.6, 114.3)
- added REF**: VIA-0.4, Dizzy:VIA-0.4, F.Cu at (123.8, 122.0)
- added REF**: VIA-0.4, Dizzy:VIA-0.4, F.Cu at (123.8, 123.6)
- added REF**: VIA-0.4, Dizzy:VIA-0.4, F.Cu at (123.8, 130.8)
- added REF**: VIA-0.4, Dizzy:VIA-0.4, F.Cu at (123.8, 129.2)
- added REF**: VIA-0.4, Dizzy:VIA-0.4, F.Cu at (123.8, 128.4)
- added REF**: VIA-0.4, Dizzy:VIA-0.4, F.Cu at (123.8, 130.0)
- added REF**: VIA-0.4, Dizzy:VIA-0.4, F.Cu at (123.8, 127.6)
- added REF**: VIA-0.4, Dizzy:VIA-0.4, F.Cu at (123.8, 126.8)
- added REF**: VIA-0.4, Dizzy:VIA-0.4, F.Cu at (123.8, 125.2)
- added REF**: VIA-0.4, Dizzy:VIA-0.4, F.Cu at (123.8, 124.4)
- added REF**: VIA-0.4, Dizzy:VIA-0.4, F.Cu at (101.3, 119.9)
- added REF**: VIA-0.4, Dizzy:VIA-0.4, F.Cu at (123.8, 126.0)
- added REF**: VIA-0.4, Dizzy:VIA-0.4, F.Cu at (124.3, 124.8)
- added REF**: VIA-0.4, Dizzy:VIA-0.4, F.Cu at (124.3, 124.0)
- added REF**: VIA-0.4, Dizzy:VIA-0.4, F.Cu at (124.3, 122.4)
- added REF**: VIA-0.4, Dizzy:VIA-0.4, F.Cu at (124.3, 121.6)
- added REF**: VIA-0.4, Dizzy:VIA-0.4, F.Cu at (124.3, 123.2)
- added REF**: VIA-0.4, Dizzy:VIA-0.4, F.Cu at (124.3, 120.9)
- added REF**: VIA-0.4, Dizzy:VIA-0.4, F.Cu at (124.3, 120.1)
- added REF**: VIA-0.4, Dizzy:VIA-0.4, F.Cu at (124.3, 118.5)
- added REF**: VIA-0.4, Dizzy:VIA-0.4, F.Cu at (124.3, 117.7)
- added REF**: VIA-0.4, Dizzy:VIA-0.4, F.Cu at (101.2, 122.5)
- added REF**: VIA-0.4, Dizzy:VIA-0.4, F.Cu at (124.3, 119.3)
- added REF**: VIA-0.4, Dizzy:VIA-0.4, F.Cu at (127.7, 120.5)
- added REF**: VIA-0.4, Dizzy:VIA-0.4, F.Cu at (127.7, 119.7)
- added REF**: VIA-0.4, Dizzy:VIA-0.4, F.Cu at (127.7, 118.1)
- added REF**: VIA-0.4, Dizzy:VIA-0.4, F.Cu at (127.7, 117.3)
- added REF**: VIA-0.4, Dizzy:VIA-0.4, F.Cu at (127.7, 118.9)
- added REF**: VIA-0.4, Dizzy:VIA-0.4, F.Cu at (127.7, 124.4)
- added REF**: VIA-0.4, Dizzy:VIA-0.4, F.Cu at (127.7, 123.6)
- added REF**: VIA-0.4, Dizzy:VIA-0.4, F.Cu at (127.7, 122.0)
- added REF**: VIA-0.4, Dizzy:VIA-0.4, F.Cu at (127.7, 121.2)
- added REF**: VIA-0.4, Dizzy:VIA-0.4, F.Cu at (109.9, 119.7)
- added REF**: VIA-0.4, Dizzy:VIA-0.4, F.Cu at (127.7, 122.8)
- added REF**: VIA-0.4, Dizzy:VIA-0.4, F.Cu at (127.2, 121.6)
- added REF**: VIA-0.4, Dizzy:VIA-0.4, F.Cu at (127.2, 123.2)
- added REF**: VIA-0.4, Dizzy:VIA-0.4, F.Cu at (127.2, 122.4)
- added REF**: VIA-0.4, Dizzy:VIA-0.4, F.Cu at (127.2, 124.0)
- added REF**: VIA-0.4, Dizzy:VIA-0.4, F.Cu at (127.2, 124.8)
- added REF**: VIA-0.4, Dizzy:VIA-0.4, F.Cu at (124.8, 117.3)
- added REF**: VIA-0.4, Dizzy:VIA-0.4, F.Cu at (125.2, 117.7)
- added REF**: VIA-0.4, Dizzy:VIA-0.4, F.Cu at (126.2, 117.7)
- added REF**: VIA-0.4, Dizzy:VIA-0.4, F.Cu at (126.7, 117.3)
- added REF**: VIA-0.4, Dizzy:VIA-0.4, F.Cu at (114.9, 124.5)
- added REF**: VIA-0.4, Dizzy:VIA-0.4, F.Cu at (127.2, 116.9)
- added REF**: VIA-0.4, Dizzy:VIA-0.4, F.Cu at (127.2, 117.7)
- added REF**: VIA-0.4, Dizzy:VIA-0.4, F.Cu at (127.2, 119.3)
- added REF**: VIA-0.4, Dizzy:VIA-0.4, F.Cu at (127.2, 118.5)
- added REF**: VIA-0.4, Dizzy:VIA-0.4, F.Cu at (127.2, 120.9)
- added REF**: VIA-0.4, Dizzy:VIA-0.4, F.Cu at (127.2, 120.1)
- added REF**: VIA-0.4, Dizzy:VIA-0.4, F.Cu at (126.7, 120.5)
- added REF**: VIA-0.4, Dizzy:VIA-0.4, F.Cu at (124.8, 120.5)
- added REF**: VIA-0.4, Dizzy:VIA-0.4, F.Cu at (125.8, 107.9)
- added REF**: VIA-0.4, Dizzy:VIA-0.4, F.Cu at (142.7, 113.7)
- added REF**: VIA-0.4, Dizzy:VIA-0.4, F.Cu at (125.8, 108.7)
- added REF**: VIA-0.4, Dizzy:VIA-0.4, F.Cu at (125.8, 109.5)
- added REF**: VIA-0.4, Dizzy:VIA-0.4, F.Cu at (125.8, 110.3)
- added REF**: VIA-0.4, Dizzy:VIA-0.4, F.Cu at (125.8, 111.1)
- added REF**: VIA-0.4, Dizzy:VIA-0.4, F.Cu at (125.8, 111.9)
- added REF**: VIA-0.4, Dizzy:VIA-0.4, F.Cu at (125.8, 112.7)
- added REF**: VIA-0.4, Dizzy:VIA-0.4, F.Cu at (125.8, 113.5)
- added REF**: VIA-0.4, Dizzy:VIA-0.4, F.Cu at (125.8, 114.3)
- added REF**: VIA-0.4, Dizzy:VIA-0.4, F.Cu at (124.9, 107.9)
- added REF**: VIA-0.4, Dizzy:VIA-0.4, F.Cu at (124.9, 108.7)
- added REF**: VIA-0.4, Dizzy:VIA-0.4, F.Cu at (119.9, 91.8)
- added REF**: VIA-0.4, Dizzy:VIA-0.4, F.Cu at (124.9, 109.5)
- added REF**: VIA-0.4, Dizzy:VIA-0.4, F.Cu at (124.9, 110.3)
- added REF**: VIA-0.4, Dizzy:VIA-0.4, F.Cu at (124.9, 111.1)
- added REF**: VIA-0.4, Dizzy:VIA-0.4, F.Cu at (124.9, 111.9)
- added REF**: VIA-0.4, Dizzy:VIA-0.4, F.Cu at (124.9, 112.7)
- added REF**: VIA-0.4, Dizzy:VIA-0.4, F.Cu at (124.9, 113.5)
- added REF**: VIA-0.4, Dizzy:VIA-0.4, F.Cu at (124.9, 114.3)
- added REF**: VIA-0.4, Dizzy:VIA-0.4, F.Cu at (124.1, 107.9)
- added REF**: VIA-0.4, Dizzy:VIA-0.4, F.Cu at (124.1, 108.7)
- added REF**: VIA-0.4, Dizzy:VIA-0.4, F.Cu at (124.1, 109.5)
- added REF**: VIA-0.4, Dizzy:VIA-0.4, F.Cu at (133.4, 98.2)
- added REF**: VIA-0.4, Dizzy:VIA-0.4, F.Cu at (124.1, 110.3)
- added REF**: VIA-0.4, Dizzy:VIA-0.4, F.Cu at (124.1, 111.1)
- added REF**: VIA-0.4, Dizzy:VIA-0.4, F.Cu at (124.1, 111.9)
- added REF**: VIA-0.4, Dizzy:VIA-0.4, F.Cu at (124.1, 112.7)
- added REF**: VIA-0.4, Dizzy:VIA-0.4, F.Cu at (124.1, 113.5)
- added REF**: VIA-0.4, Dizzy:VIA-0.4, F.Cu at (124.1, 114.3)
- added REF**: VIA-0.4, Dizzy:VIA-0.4, F.Cu at (123.3, 107.9)
- added REF**: VIA-0.4, Dizzy:VIA-0.4, F.Cu at (123.3, 108.7)
- added REF**: VIA-0.4, Dizzy:VIA-0.4, F.Cu at (123.3, 109.5)
- added REF**: VIA-0.4, Dizzy:VIA-0.4, F.Cu at (123.3, 110.3)
- added REF**: VIA-0.4, Dizzy:VIA-0.4, F.Cu at (131.4, 101.7)
- added REF**: VIA-0.4, Dizzy:VIA-0.4, F.Cu at (123.3, 111.1)
- added REF**: VIA-0.4, Dizzy:VIA-0.4, F.Cu at (123.3, 111.9)
- added REF**: VIA-0.4, Dizzy:VIA-0.4, F.Cu at (123.3, 112.7)
- added REF**: VIA-0.4, Dizzy:VIA-0.4, F.Cu at (123.3, 113.5)
- added REF**: VIA-0.4, Dizzy:VIA-0.4, F.Cu at (123.3, 114.3)
- added REF**: VIA-0.4, Dizzy:VIA-0.4, F.Cu at (122.5, 107.9)
- added REF**: VIA-0.4, Dizzy:VIA-0.4, F.Cu at (122.5, 108.7)
- added REF**: VIA-0.4, Dizzy:VIA-0.4, F.Cu at (122.5, 109.5)
- added REF**: VIA-0.4, Dizzy:VIA-0.4, F.Cu at (122.5, 110.3)
- added REF**: VIA-0.4, Dizzy:VIA-0.4, F.Cu at (122.5, 111.9)
- added REF**: VIA-0.4, Dizzy:VIA-0.4, F.Cu at (114.6, 104.7)
- added REF**: VIA-0.4, Dizzy:VIA-0.4, F.Cu at (122.5, 112.7)
- added REF**: VIA-0.4, Dizzy:VIA-0.4, F.Cu at (122.5, 113.5)
- added REF**: VIA-0.4, Dizzy:VIA-0.4, F.Cu at (122.5, 114.3)
- added REF**: VIA-0.4, Dizzy:VIA-0.4, F.Cu at (121.7, 107.9)
- added REF**: VIA-0.4, Dizzy:VIA-0.4, F.Cu at (121.7, 108.7)
- added REF**: VIA-0.4, Dizzy:VIA-0.4, F.Cu at (121.7, 109.5)
- added REF**: VIA-0.4, Dizzy:VIA-0.4, F.Cu at (121.7, 110.3)
- added REF**: VIA-0.4, Dizzy:VIA-0.4, F.Cu at (121.7, 111.1)
- added REF**: VIA-0.4, Dizzy:VIA-0.4, F.Cu at (121.7, 111.9)
- added REF**: VIA-0.4, Dizzy:VIA-0.4, F.Cu at (121.7, 112.7)
- added REF**: VIA-0.4, Dizzy:VIA-0.4, F.Cu at (112.2, 102.3)
- added REF**: VIA-0.4, Dizzy:VIA-0.4, F.Cu at (121.7, 113.5)
- added REF**: VIA-0.4, Dizzy:VIA-0.4, F.Cu at (121.7, 114.3)
- added REF**: VIA-0.4, Dizzy:VIA-0.4, F.Cu at (120.9, 107.9)
- added REF**: VIA-0.4, Dizzy:VIA-0.4, F.Cu at (120.9, 108.7)
- added REF**: VIA-0.4, Dizzy:VIA-0.4, F.Cu at (120.9, 109.5)
- added REF**: VIA-0.4, Dizzy:VIA-0.4, F.Cu at (120.9, 110.3)
- added REF**: VIA-0.4, Dizzy:VIA-0.4, F.Cu at (120.9, 111.1)
- added REF**: VIA-0.4, Dizzy:VIA-0.4, F.Cu at (120.9, 111.9)
- added REF**: VIA-0.4, Dizzy:VIA-0.4, F.Cu at (120.9, 112.7)
- added REF**: VIA-0.4, Dizzy:VIA-0.4, F.Cu at (120.9, 113.5)
- added REF**: VIA-0.4, Dizzy:VIA-0.4, F.Cu at (102.1, 95.1)
- added REF**: VIA-0.4, Dizzy:VIA-0.4, F.Cu at (120.9, 114.3)
- added REF**: VIA-0.4, Dizzy:VIA-0.4, F.Cu at (119.3, 114.3)
- added REF**: VIA-0.4, Dizzy:VIA-0.4, F.Cu at (119.3, 113.5)
- added REF**: VIA-0.4, Dizzy:VIA-0.4, F.Cu at (119.3, 112.7)
- added REF**: VIA-0.4, Dizzy:VIA-0.4, F.Cu at (120.1, 114.3)
- added REF**: VIA-0.4, Dizzy:VIA-0.4, F.Cu at (120.1, 111.1)
- added REF**: VIA-0.4, Dizzy:VIA-0.4, F.Cu at (120.1, 111.9)
- added REF**: VIA-0.4, Dizzy:VIA-0.4, F.Cu at (120.1, 110.3)
- added REF**: VIA-0.4, Dizzy:VIA-0.4, F.Cu at (120.1, 113.5)
- added REF**: VIA-0.4, Dizzy:VIA-0.4, F.Cu at (120.1, 112.7)
- added REF**: VIA-0.4, Dizzy:VIA-0.4, F.Cu at (98.9, 95.0)
- added REF**: VIA-0.4, Dizzy:VIA-0.4, F.Cu at (119.3, 111.9)
- added REF**: VIA-0.4, Dizzy:VIA-0.4, F.Cu at (119.3, 108.7)
- added REF**: VIA-0.4, Dizzy:VIA-0.4, F.Cu at (119.3, 109.5)
- added REF**: VIA-0.4, Dizzy:VIA-0.4, F.Cu at (119.3, 107.9)
- added REF**: VIA-0.4, Dizzy:VIA-0.4, F.Cu at (119.3, 111.1)
- added REF**: VIA-0.4, Dizzy:VIA-0.4, F.Cu at (119.3, 110.3)
- added REF**: VIA-0.4, Dizzy:VIA-0.4, F.Cu at (122.3, 131.2)
- added REF**: VIA-0.4, Dizzy:VIA-0.4, F.Cu at (122.8, 130.8)
- added REF**: VIA-0.4, Dizzy:VIA-0.4, F.Cu at (131.7, 131.3)
- added REF**: VIA-0.4, Dizzy:VIA-0.4, F.Cu at (123.3, 127.2)
- U3: footprint Housings_QFP:TQFP-64-1EP_10x10mm_Pitch0.5mm -> Housings_DFN_QFN:QFN-64-1EP_9x9mm_Pitch0.5mm
Connections:
- J5 pad 2: 3v3 -> FLASH_TX
- J5 pad 3: GPIO0 -> nRESET
- J5 pad 4: GPIO4 -> FLASH_RX
- J5 pad 5: GPIO5 -> GPIO6
- J5 pad 6: GPIO6 -> GPIO7
- J5 pad 7: GPIO7 -> 3v3
- U3 pad 50: GPIO0 -> Net-(U3-Pad50)
- U3 pad 55: Net-(U3-Pad55) -> FLASH_TX
- U3 pad 57: ADC_V -> FLASH_RX
- U3 pad 59: GPIO4 -> ADC_V
- U3 pad 60: GPIO5 -> Net-(U3-Pad60)
Routing:
- net 3v3: track 138.1 -> 173.7 mm
- net nRESET: track 27.6 -> 63.2 mm
- net GPIO0: track 17.8 -> 0.00 mm, vias 2 -> 0
- net FLASH_TX: track 0.00 -> 15.6 mm
- net FLASH_RX: track 0.00 -> 12.9 mm
- net GPIO5: track 12.5 -> 0.00 mm
- net GPIO4: track 11.0 -> 0.00 mm
- net GPIO8: track 12.7 -> 6.31 mm
- net GPIO6: track 8.01 -> 13.6 mm
- net VDD_DIG: track 42.9 -> 46.6 mm, vias 0 -> 6
- net VDD_ANA: track 50.6 -> 54.3 mm, vias 0 -> 4
- net VDD_PA: track 23.3 -> 25.9 mm, vias 3 -> 5
- net ADC_I: track 14.2 -> 16.5 mm, vias 0 -> 2
- net GPIO7: track 7.07 -> 9.06 mm
- net (no net): track 0.00 -> 1.92 mm
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Other:
- board text added: "3v3"
- board text added: "A"
- board text added: "B"
- board text added: "GND"
- board text added: "GPIO6"
- board text added: "GPIO7"
- board text added: "GPIO8"
- board text added: "JTAG"
- board text added: "RESET"
- board text added: "RS485"
- board text added: "RX"
- board text added: "TX"
