File: Schamatic/Mainboard/Mainboard.kicad_pcb (KiCad board)
At the start: 4 copper layers, 60.3 x 55.7 mm, 288 parts, among them J1 BAT+, J10 BAT-, J11 PLUG+, J12 PLUG-, J13 MOUNT, J14 MOUNT, J15 MOUNT, J16 MOUNT, J2 M+1, J3 USART, J4 3.3V, J5 CONN_02X04, J6 JTAG, J7 M+2, J8 M-1, J9 M-2, Q1 p-MOSFET, SW1 B3U-1000P, SW2 B3U-1000P, SW3 B3U-1000P, SW4 B3U-1000P, SW5 B3U-1000P, U1 ACS781, U2 ADP2303ARDZ-3.3, U3 cc3220, U4 DEA202450BT-3201B2, U5 MX25R3235F, U6 LSM9DS1, U7 LTC2954, U8 LTC2876, Y1 32.768kHz, Y2 40Mhz

Commit message: SolidWorks 3D
Routing:
- net Earth: track 31.8 -> 33.7 mm, vias 56 -> 55
- net (no net): track 1.92 -> 0.00 mm
- net 12V: track 49.1 -> 49.8 mm
Changed lines of the file:
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@@
 (kicad_pcb (version 4) (host pcbnew 4.0.6)
   (general
-    (links 258)
+    (links 445)
     (no_connects 0)
     (area 88.744999 74.545 150.053 134.205)
@@
   )
   (setup
-    (last_trace_width 0.25)
+    (last_trace_width 0.13)
     (user_trace_width 0.13)
     (user_trace_width 0.25)
@@
     (mod_text_size 1 1)
     (mod_text_width 0.15)
-    (pad_size 0.4 0.4)
-    (pad_drill 0.25)
+    (pad_size 3.5 3.5)
+    (pad_drill 2)
     (pad_to_mask_clearance 0.2)
     (aux_axis_origin 0 0)
@@
     (fp_circle (center 0 0) (end 2.6 0) (layer F.CrtYd) (width 0.05))
     (fp_circle (center 0 0) (end 0 -2.286) (layer F.SilkS) (width 0.12))
-    (pad 1 thru_hole circle (at 0 0) (size 3.5 3.5) (drill 2.2) (layers *.Cu *.Mask)
+    (pad 1 thru_hole circle (at 0 0) (size 3.5 3.5) (drill 2) (layers *.Cu *.Mask)
       (net 72 "Net-(J2-Pad1)") (zone_connect 2))
   )
@@
     (fp_circle (center 0 0) (end 2.6 0) (layer F.CrtYd) (width 0.05))
     (fp_circle (center 0 0) (end 0 -2.286) (layer F.SilkS) (width 0.12))
-    (pad 1 thru_hole circle (at 0 0) (size 3.5 3.5) (drill 2.2) (layers *.Cu *.Mask)
+    (pad 1 thru_hole circle (at 0 0) (size 3.5 3.5) (drill 2) (layers *.Cu *.Mask)
       (net 72 "Net-(J2-Pad1)") (zone_connect 2))
   )
@@
     (fp_circle (center 0 0) (end 2.6 0) (layer F.CrtYd) (width 0.05))
     (fp_circle (center 0 0) (end 0 -2.286) (layer F.SilkS) (width 0.12))
-    (pad 1 thru_hole circle (at 0 0) (size 3.5 3.5) (drill 2.2) (layers *.Cu *.Mask)
+    (pad 1 thru_hole circle (at 0 0) (size 3.5 3.5) (drill 2) (layers *.Cu *.Mask)
       (net 1 Earth) (zone_connect 2))
   )
@@
     (fp_circle (center 0 0) (end 2.6 0) (layer F.CrtYd) (width 0.05))
     (fp_circle (center 0 0) (end 0 -2.286) (layer F.SilkS) (width 0.12))
-    (pad 1 thru_hole circle (at 0 0 180) (size 3.5 3.5) (drill 2.2) (layers *.Cu *.Mask)
+    (pad 1 thru_hole circle (at 0 0 180) (size 3.5 3.5) (drill 2) (layers *.Cu *.Mask)
       (net 1 Earth) (zone_connect 2))
   )
@@
     (fp_circle (center 0 0) (end 2.6 0) (layer F.CrtYd) (width 0.05))
     (fp_circle (center 0 0) (end 0 -2.286) (layer F.SilkS) (width 0.12))
-    (pad 1 thru_hole circle (at 0 0 180) (size 3.5 3.5) (drill 2.2) (layers *.Cu *.Mask)
+    (pad 1 thru_hole circle (at 0 0 180) (size 3.5 3.5) (drill 2) (layers *.Cu *.Mask)
       (net 1 Earth) (zone_connect 2))
   )
@@
     (fp_circle (center 0 0) (end 2.6 0) (layer F.CrtYd) (width 0.05))
     (fp_circle (center 0 0) (end 0 -2.286) (layer F.SilkS) (width 0.12))
-    (pad 1 thru_hole circle (at 0 0) (size 4.064 4.064) (drill 3.048) (layers *.Cu *.Mask)
+    (pad 1 thru_hole circle (at 0 0) (size 3.5 3.5) (drill 2) (layers *.Cu *.Mask)
       (net 1 Earth))
   )
@@
   (gr_line (start 149.4 76.6) (end 149.4 132.200089) (layer Edge.Cuts) (width 0.15))
   (gr_line (start 89.099823 132.25) (end 149.400186 132.25) (layer Edge.Cuts) (width 0.15))
-  (segment (start 126.625 120.525) (end 124.7 120.525) (width 0.25) (layer F.Cu) (net 0))
-  (via (at 118.820685 121.020685) (size 0.4) (drill 0.25) (layers F.Cu B.Cu) (net 1))
+  (segment (start 126.625 120.525) (end 124.7 120.525) (width 0.25) (layer F.Cu) (net 1))
   (segment (start 126.75 121) (end 127.275 121) (width 0.25) (layer F.Cu) (net 1))
   (segment (start 126.75 120.05) (end 126.75 119.575) (width 0.25) (layer F.Cu) (net 1))
@@
   (via (at 123.6 100.9) (size 0.4) (drill 0.25) (layers F.Cu B.Cu) (net 1) (status 30))
   (via (at 122 100.9) (size 0.4) (drill 0.25) (layers F.Cu B.Cu) (net 1) (status 30))
+  (segment (start 124.8 85.7) (end 124.8 84.3) (width 0.5) (layer F.Cu) (net 2))
+  (segment (start 124.8 84.3) (end 124.4 83.9) (width 0.5) (layer F.Cu) (net 2))
+  (segment (start 124.3 79.2) (end 123.6 79.2) (width 0.5) (layer F.Cu) (net 2))
+  (segment (start 124.4 83.9) (end 124.4 79.3) (width 0.5) (layer F.Cu) (net 2))
+  (segment (start 124.4 79.3) (end 124.3 79.2) (width 0.5) (layer F.Cu) (net 2))
+  (segment (start 123.6 79.2) (end 123.6 78.3) (width 0.5) (layer F.Cu) (net 2))
+  (segment (start 123.6 78.3) (end 122.5 77.2) (width 0.5) (layer F.Cu) (net 2))
+  (segment (start 122.5 77.2) (end 107.15 77.2) (width 0.5) (layer F.Cu) (net 2))
+  (segment (start 107.15 77.2) (end 106.180001 78.169999) (width 0.5) (layer F.Cu) (net 2))
   (segment (start 105 78.6) (end 105 77.9) (width 0.25) (layer F.Cu) (net 2) (status 10))
   (segment (start 105 77.9) (end 104.994999 77.894999) (width 0.25) (layer F.Cu) (net 2))
@@
   (segment (start 106.180001 81.738591) (end 106.180001 78.169999) (width 0.5) (layer F.Cu) (net 2))
   (segment (start 104.88511 81.758482) (end 104.88511 83.028482) (width 0.5) (layer F.Cu) (net 2) (status 30))
-  (segment (start 123.6 79.2) (end 123.6 78.3) (width 0.5) (layer F.Cu) (net 2) (status 10))
-  (segment (start 123.6 78.3) (end 123.469999 78.169999) (width 0.5) (layer F.Cu) (net 2))
   (segment (start 105.75 78.6) (end 105 78.6) (width 0.5) (layer F.Cu) (net 2) (status 20))
-  (segment (start 123.469999 78.169999) (end 106.180001 78.169999) (width 0.5) (layer F.Cu) (net 2))
   (segment (start 106.180001 78.169999) (end 105.75 78.6) (width 0.5) (layer F.Cu) (net 2))
-  (segment (start 124.8 85.7) (end 124.8 84.3) (width 0.5) (layer F.Cu) (net 2) (status 10))
-  (segment (start 124.8 84.3) (end 124.569999 84.069999) (width 0.5) (layer F.Cu) (net 2))
-  (segment (start 124.569999 84.069999) (end 124.569999 79.269999) (width 0.5) (layer F.Cu) (net 2))
-  (segment (start 124.569999 79.269999) (end 124.5 79.2) (width 0.5) (layer F.Cu) (net 2))
-  (segment (start 124.5 79.2) (end 123.6 79.2) (width 0.5) (layer F.Cu) (net 2) (status 20))
   (segment (start 129.7 88.9) (end 129.7 92.4) (width 0.25) (layer F.Cu) (net 2) (status 10))
   (segment (start 129.7 92.4) (end 128.7 93.4) (width 0.25) (layer F.Cu) (net 2) (status 20))

Commit message: motherboard corrections
Parts:
- removed the REF** at (119.3, 129.0)
- removed the REF** at (98.7, 101.1)
- removed the REF** at (123.3, 126.4)
- removed the REF** at (123.3, 129.6)
- removed the REF** at (123.3, 130.4)
- removed the REF** at (131.2, 126.7)
- removed the REF** at (131.2, 127.7)
- removed the REF** at (131.2, 130.9)
- removed the REF** at (130.7, 129.7)
- removed the REF** at (91.1, 107.4)
- removed the REF** at (131.2, 129.3)
- removed the REF** at (131.2, 128.5)
- removed the REF** at (131.2, 130.1)
- removed the REF** at (130.7, 128.1)
- removed the REF** at (130.7, 127.3)
- removed the REF** at (130.5, 126.6)
- removed the REF** at (130.1, 126.1)
- removed the REF** at (129.7, 126.6)
- removed the REF** at (129.3, 126.1)
- removed the REF** at (90.7, 117.0)
- removed the REF** at (128.9, 126.6)
- removed the REF** at (128.1, 126.6)
- removed the REF** at (128.5, 126.1)
- removed the REF** at (128.5, 125.2)
- removed the REF** at (128.1, 125.7)
- removed the REF** at (127.7, 125.2)
- removed the REF** at (124.3, 126.4)
- removed the REF** at (124.3, 125.6)
- removed the REF** at (124.8, 121.3)
- removed the REF** at (126.7, 121.3)
- removed the REF** at (98.4, 114.0)
- removed the REF** at (126.7, 118.1)
- removed the REF** at (126.7, 118.9)
- removed the REF** at (124.8, 118.0)
- removed the REF** at (124.8, 118.9)
- removed the REF** at (123.7, 118.1)
- removed the REF** at (123.7, 118.9)
- removed the REF** at (123.7, 120.4)
- removed the REF** at (123.7, 119.6)
- removed the REF** at (123.7, 121.2)
- removed the REF** at (123.8, 122.8)
- removed the REF** at (106.6, 114.3)
- removed the REF** at (123.8, 122.0)
- removed the REF** at (123.8, 123.6)
- removed the REF** at (123.8, 130.8)
- removed the REF** at (123.8, 129.2)
- removed the REF** at (123.8, 128.4)
- removed the REF** at (123.8, 130.0)
- removed the REF** at (123.8, 127.6)
- removed the REF** at (123.8, 126.8)
- removed the REF** at (123.8, 125.2)
- removed the REF** at (123.8, 124.4)
- removed the REF** at (101.3, 119.9)
- removed the REF** at (123.8, 126.0)
- removed the REF** at (124.3, 124.8)
- removed the REF** at (124.3, 124.0)
- removed the REF** at (124.3, 122.4)
- removed the REF** at (124.3, 121.6)
- removed the REF** at (124.3, 123.2)
- removed the REF** at (124.3, 120.9)
- removed the REF** at (124.3, 120.1)
- removed the REF** at (124.3, 118.5)
- removed the REF** at (124.3, 117.7)
- removed the REF** at (101.2, 122.5)
- removed the REF** at (124.3, 119.3)
- removed the REF** at (127.7, 120.5)
- removed the REF** at (127.7, 119.7)
- removed the REF** at (127.7, 118.1)
- removed the REF** at (127.7, 117.3)
- removed the REF** at (127.7, 118.9)
- removed the REF** at (127.7, 124.4)
- removed the REF** at (127.7, 123.6)
- removed the REF** at (127.7, 122.0)
- removed the REF** at (127.7, 121.2)
- removed the REF** at (109.9, 119.7)
- removed the REF** at (127.7, 122.8)
- removed the REF** at (127.2, 121.6)
- removed the REF** at (127.2, 123.2)
- removed the REF** at (127.2, 122.4)
- removed the REF** at (127.2, 124.0)
- removed the REF** at (127.2, 124.8)
- removed the REF** at (124.8, 117.3)
- removed the REF** at (125.2, 117.7)
- removed the REF** at (126.2, 117.7)
- removed the REF** at (126.7, 117.3)
- removed the REF** at (114.9, 124.5)
- removed the REF** at (127.2, 116.9)
- removed the REF** at (127.2, 117.7)
- removed the REF** at (127.2, 119.3)
- removed the REF** at (127.2, 118.5)
- removed the REF** at (127.2, 120.9)
- removed the REF** at (127.2, 120.1)
- removed the REF** at (126.7, 120.5)
- removed the REF** at (124.8, 120.5)
- removed the REF** at (125.8, 107.9)
- removed the REF** at (142.7, 113.7)
- removed the REF** at (125.8, 108.7)
- removed the REF** at (125.8, 109.5)
- removed the REF** at (125.8, 110.3)
- removed the REF** at (125.8, 111.1)
- removed the REF** at (125.8, 111.9)
- removed the REF** at (125.8, 112.7)
- removed the REF** at (125.8, 113.5)
- removed the REF** at (125.8, 114.3)
- removed the REF** at (124.9, 107.9)
- removed the REF** at (124.9, 108.7)
- removed the REF** at (119.9, 91.8)
- removed the REF** at (124.9, 109.5)
- removed the REF** at (124.9, 110.3)
- removed the REF** at (124.9, 111.1)
- removed the REF** at (124.9, 111.9)
- removed the REF** at (124.9, 112.7)
- removed the REF** at (124.9, 113.5)
- removed the REF** at (124.9, 114.3)
- removed the REF** at (124.1, 107.9)
- removed the REF** at (124.1, 108.7)
- removed the REF** at (124.1, 109.5)
- removed the REF** at (133.4, 98.2)
- removed the REF** at (124.1, 110.3)
- removed the REF** at (124.1, 111.1)
- removed the REF** at (124.1, 111.9)
- removed the REF** at (124.1, 112.7)
- removed the REF** at (124.1, 113.5)
- removed the REF** at (124.1, 114.3)
- removed the REF** at (123.3, 107.9)
- removed the REF** at (123.3, 108.7)
- removed the REF** at (123.3, 109.5)
- removed the REF** at (123.3, 110.3)
- removed the REF** at (131.4, 101.7)
- removed the REF** at (123.3, 111.1)
- removed the REF** at (123.3, 111.9)
- removed the REF** at (123.3, 112.7)
- removed the REF** at (123.3, 113.5)
- removed the REF** at (123.3, 114.3)
- removed the REF** at (122.5, 107.9)
- removed the REF** at (122.5, 108.7)
- removed the REF** at (122.5, 109.5)
- removed the REF** at (122.5, 110.3)
- removed the REF** at (122.5, 111.9)
- removed the REF** at (114.6, 104.7)
- removed the REF** at (122.5, 112.7)
- removed the REF** at (122.5, 113.5)
- removed the REF** at (122.5, 114.3)
- removed the REF** at (121.7, 107.9)
- removed the REF** at (121.7, 108.7)
- removed the REF** at (121.7, 109.5)
- removed the REF** at (121.7, 110.3)
- removed the REF** at (121.7, 111.1)
- removed the REF** at (121.7, 111.9)
- removed the REF** at (121.7, 112.7)
- removed the REF** at (112.2, 102.3)
- removed the REF** at (121.7, 113.5)
- removed the REF** at (121.7, 114.3)
- removed the REF** at (120.9, 107.9)
- removed the REF** at (120.9, 108.7)
- removed the REF** at (120.9, 109.5)
- removed the REF** at (120.9, 110.3)
- removed the REF** at (120.9, 111.1)
- removed the REF** at (120.9, 111.9)
- removed the REF** at (120.9, 112.7)
- removed the REF** at (120.9, 113.5)
- removed the REF** at (102.1, 95.1)
- removed the REF** at (120.9, 114.3)
- removed the REF** at (119.3, 114.3)
- removed the REF** at (119.3, 113.5)
- removed the REF** at (119.3, 112.7)
- removed the REF** at (120.1, 114.3)
- removed the REF** at (120.1, 111.1)
- removed the REF** at (120.1, 111.9)
- removed the REF** at (120.1, 110.3)
- removed the REF** at (120.1, 113.5)
- removed the REF** at (120.1, 112.7)
- removed the REF** at (98.9, 95.0)
- removed the REF** at (119.3, 111.9)
- removed the REF** at (119.3, 108.7)
- removed the REF** at (119.3, 109.5)
- removed the REF** at (119.3, 107.9)
- removed the REF** at (119.3, 111.1)
- removed the REF** at (119.3, 110.3)
- removed the REF** at (122.3, 131.2)
- removed the REF** at (122.8, 130.8)
- removed the REF** at (131.7, 131.3)
- removed the REF** at (123.3, 127.2)
- added R20: 100K, Resistors_SMD:R_0603, F.Cu at (136.7, 119.2)
- added R21: 270, Resistors_SMD:R_0603, F.Cu at (136.8, 122.0)
- added R22: 2.7K, Resistors_SMD:R_0603, F.Cu at (119.7, 119.3)
- added REF**: VIA-0.4, Dizzy:VIA-0.4, F.Cu at (129.9, 126.3)
- added REF**: VIA-0.4, Dizzy:VIA-0.4, F.Cu at (127.5, 119.0)
- added REF**: VIA-0.4, Dizzy:VIA-0.4, F.Cu at (124.6, 125.6)
- added REF**: VIA-0.4, Dizzy:VIA-0.4, F.Cu at (124.6, 126.2)
- added REF**: VIA-0.4, Dizzy:VIA-0.4, F.Cu at (124.6, 126.8)
- added REF**: VIA-0.4, Dizzy:VIA-0.4, F.Cu at (124.0, 128.2)
- added REF**: VIA-0.4, Dizzy:VIA-0.4, F.Cu at (124.0, 128.8)
- added REF**: VIA-0.4, Dizzy:VIA-0.4, F.Cu at (124.0, 129.4)
- added REF**: VIA-0.4, Dizzy:VIA-0.4, F.Cu at (124.0, 130.0)
- added REF**: VIA-0.4, Dizzy:VIA-0.4, F.Cu at (124.0, 130.6)
- added REF**: VIA-0.4, Dizzy:VIA-0.4, F.Cu at (124.0, 131.2)
- added REF**: VIA-0.4, Dizzy:VIA-0.4, F.Cu at (127.5, 120.2)
- added REF**: VIA-0.4, Dizzy:VIA-0.4, F.Cu at (127.5, 122.0)
- added REF**: VIA-0.4, Dizzy:VIA-0.4, F.Cu at (127.5, 122.6)
- added REF**: VIA-0.4, Dizzy:VIA-0.4, F.Cu at (127.5, 123.3)
- added REF**: VIA-0.4, Dizzy:VIA-0.4, F.Cu at (127.5, 126.3)
- added REF**: VIA-0.4, Dizzy:VIA-0.4, F.Cu at (127.5, 124.5)
- added REF**: VIA-0.4, Dizzy:VIA-0.4, F.Cu at (127.5, 125.7)
- added REF**: VIA-0.4, Dizzy:VIA-0.4, F.Cu at (127.5, 123.9)
- added REF**: VIA-0.4, Dizzy:VIA-0.4, F.Cu at (127.5, 125.1)
- added REF**: VIA-0.4, Dizzy:VIA-0.4, F.Cu at (129.3, 126.3)
- added REF**: VIA-0.4, Dizzy:VIA-0.4, F.Cu at (131.3, 127.0)
- added REF**: VIA-0.4, Dizzy:VIA-0.4, F.Cu at (131.3, 127.6)
- added REF**: VIA-0.4, Dizzy:VIA-0.4, F.Cu at (131.3, 128.3)
- added REF**: VIA-0.4, Dizzy:VIA-0.4, F.Cu at (131.3, 131.3)
- added REF**: VIA-0.4, Dizzy:VIA-0.4, F.Cu at (131.3, 129.5)
- added REF**: VIA-0.4, Dizzy:VIA-0.4, F.Cu at (131.3, 130.7)
- added REF**: VIA-0.4, Dizzy:VIA-0.4, F.Cu at (131.3, 128.9)
- added REF**: VIA-0.4, Dizzy:VIA-0.4, F.Cu at (131.3, 130.1)
- added REF**: VIA-0.4, Dizzy:VIA-0.4, F.Cu at (123.3, 127.4)
- added REF**: VIA-0.4, Dizzy:VIA-0.4, F.Cu at (123.3, 125.6)
- added REF**: VIA-0.4, Dizzy:VIA-0.4, F.Cu at (128.7, 126.3)
- added REF**: VIA-0.4, Dizzy:VIA-0.4, F.Cu at (123.3, 126.8)
- added REF**: VIA-0.4, Dizzy:VIA-0.4, F.Cu at (123.3, 126.2)
- added REF**: VIA-0.4, Dizzy:VIA-0.4, F.Cu at (123.3, 129.4)
- added REF**: VIA-0.4, Dizzy:VIA-0.4, F.Cu at (123.3, 130.0)
- added REF**: VIA-0.4, Dizzy:VIA-0.4, F.Cu at (123.3, 130.6)
- added REF**: VIA-0.4, Dizzy:VIA-0.4, F.Cu at (123.9, 119.9)
- added REF**: VIA-0.4, Dizzy:VIA-0.4, F.Cu at (123.9, 121.9)
- added REF**: VIA-0.4, Dizzy:VIA-0.4, F.Cu at (128.1, 126.3)
- added REF**: VIA-0.4, Dizzy:VIA-0.4, F.Cu at (123.9, 120.7)
- added REF**: VIA-0.4, Dizzy:VIA-0.4, F.Cu at (123.9, 121.3)
- added REF**: VIA-0.4, Dizzy:VIA-0.4, F.Cu at (123.9, 119.3)
- added REF**: VIA-0.4, Dizzy:VIA-0.4, F.Cu at (123.9, 118.7)
- added REF**: VIA-0.4, Dizzy:VIA-0.4, F.Cu at (124.0, 123.6)
- added REF**: VIA-0.4, Dizzy:VIA-0.4, F.Cu at (124.0, 125.6)
- added REF**: VIA-0.4, Dizzy:VIA-0.4, F.Cu at (124.0, 124.4)
- added REF**: VIA-0.4, Dizzy:VIA-0.4, F.Cu at (124.0, 125.0)
- added REF**: VIA-0.4, Dizzy:VIA-0.4, F.Cu at (124.0, 123.0)
- added REF**: VIA-0.4, Dizzy:VIA-0.4, F.Cu at (124.0, 122.4)
- added REF**: VIA-0.4, Dizzy:VIA-0.4, F.Cu at (127.5, 117.7)
- added REF**: VIA-0.4, Dizzy:VIA-0.4, F.Cu at (129.9, 126.8)
- added REF**: VIA-0.4, Dizzy:VIA-0.4, F.Cu at (129.3, 126.8)
- added REF**: VIA-0.4, Dizzy:VIA-0.4, F.Cu at (128.7, 126.8)
- added REF**: VIA-0.4, Dizzy:VIA-0.4, F.Cu at (128.1, 126.8)
- added REF**: VIA-0.4, Dizzy:VIA-0.4, F.Cu at (127.5, 126.8)
- added REF**: VIA-0.4, Dizzy:VIA-0.4, F.Cu at (124.6, 117.5)
- added REF**: VIA-0.4, Dizzy:VIA-0.4, F.Cu at (126.9, 117.6)
- added REF**: VIA-0.4, Dizzy:VIA-0.4, F.Cu at (126.3, 117.6)
- added REF**: VIA-0.4, Dizzy:VIA-0.4, F.Cu at (126.3, 117.0)
- added REF**: VIA-0.4, Dizzy:VIA-0.4, F.Cu at (125.2, 117.0)
- added REF**: VIA-0.4, Dizzy:VIA-0.4, F.Cu at (127.5, 118.4)
- added REF**: VIA-0.4, Dizzy:VIA-0.4, F.Cu at (125.2, 117.6)
- added REF**: VIA-0.4, Dizzy:VIA-0.4, F.Cu at (124.6, 118.7)
- added REF**: VIA-0.4, Dizzy:VIA-0.4, F.Cu at (124.6, 118.1)
- added REF**: VIA-0.4, Dizzy:VIA-0.4, F.Cu at (124.6, 119.3)
- added REF**: VIA-0.4, Dizzy:VIA-0.4, F.Cu at (126.9, 118.9)
- added REF**: VIA-0.4, Dizzy:VIA-0.4, F.Cu at (126.9, 118.3)
- added REF**: VIA-0.4, Dizzy:VIA-0.4, F.Cu at (126.9, 119.5)
- added REF**: VIA-0.4, Dizzy:VIA-0.4, F.Cu at (124.0, 126.8)
- added REF**: VIA-0.4, Dizzy:VIA-0.4, F.Cu at (124.0, 126.2)
- added REF**: VIA-0.4, Dizzy:VIA-0.4, F.Cu at (124.0, 127.4)
- added REF**: VIA-0.4, Dizzy:VIA-0.4, F.Cu at (127.5, 121.4)
- added REF**: VIA-0.4, Dizzy:VIA-0.4, F.Cu at (130.7, 126.4)
- added REF**: VIA-0.4, Dizzy:VIA-0.4, F.Cu at (130.7, 127.0)
- added REF**: VIA-0.4, Dizzy:VIA-0.4, F.Cu at (130.7, 127.6)
- added REF**: VIA-0.4, Dizzy:VIA-0.4, F.Cu at (130.7, 128.3)
- added REF**: VIA-0.4, Dizzy:VIA-0.4, F.Cu at (130.7, 129.5)
- added REF**: VIA-0.4, Dizzy:VIA-0.4, F.Cu at (130.7, 130.1)
- added REF**: VIA-0.4, Dizzy:VIA-0.4, F.Cu at (130.7, 130.7)
- added REF**: VIA-0.4, Dizzy:VIA-0.4, F.Cu at (130.7, 131.3)
- added REF**: VIA-0.4, Dizzy:VIA-0.4, F.Cu at (126.9, 120.2)
- added REF**: VIA-0.4, Dizzy:VIA-0.4, F.Cu at (127.5, 119.6)
- added REF**: VIA-0.4, Dizzy:VIA-0.4, F.Cu at (126.9, 120.8)
- added REF**: VIA-0.4, Dizzy:VIA-0.4, F.Cu at (126.9, 121.4)
- added REF**: VIA-0.4, Dizzy:VIA-0.4, F.Cu at (126.9, 122.0)
- added REF**: VIA-0.4, Dizzy:VIA-0.4, F.Cu at (126.9, 122.6)
- added REF**: VIA-0.4, Dizzy:VIA-0.4, F.Cu at (126.9, 123.2)
- added REF**: VIA-0.4, Dizzy:VIA-0.4, F.Cu at (126.9, 123.8)
- added REF**: VIA-0.4, Dizzy:VIA-0.4, F.Cu at (126.9, 124.4)
- added REF**: VIA-0.4, Dizzy:VIA-0.4, F.Cu at (126.9, 125.0)
- added REF**: VIA-0.4, Dizzy:VIA-0.4, F.Cu at (126.9, 125.6)
- added REF**: VIA-0.4, Dizzy:VIA-0.4, F.Cu at (126.9, 126.2)
- added REF**: VIA-0.4, Dizzy:VIA-0.4, F.Cu at (127.5, 120.8)
- added REF**: VIA-0.4, Dizzy:VIA-0.4, F.Cu at (126.9, 126.8)
- added REF**: VIA-0.4, Dizzy:VIA-0.4, F.Cu at (124.6, 120.1)
- added REF**: VIA-0.4, Dizzy:VIA-0.4, F.Cu at (124.6, 120.7)
- added REF**: VIA-0.4, Dizzy:VIA-0.4, F.Cu at (124.6, 121.3)
- added REF**: VIA-0.4, Dizzy:VIA-0.4, F.Cu at (124.6, 121.9)
- added REF**: VIA-0.4, Dizzy:VIA-0.4, F.Cu at (124.6, 122.5)
- added REF**: VIA-0.4, Dizzy:VIA-0.4, F.Cu at (124.6, 123.1)
- added REF**: VIA-0.4, Dizzy:VIA-0.4, F.Cu at (124.6, 123.8)
- added REF**: VIA-0.4, Dizzy:VIA-0.4, F.Cu at (124.6, 124.4)
- added REF**: VIA-0.4, Dizzy:VIA-0.4, F.Cu at (124.6, 125.0)
- C27: footprint Capacitors_SMD:C_0805 -> Capacitors_SMD:C_0603
- C3, C4: value 0.1uF 25V -> 0.1uF
- C5, C6: value GRM31CR60J226KE19 -> 22uF
- R10, R11, R12, R9: value 300 -> 470
- R6: value 1.2k -> 2k
- moved J13 5.65 mm to (140.1, 128.9)
- moved J15 5.60 mm to (140.4, 79.8)
- moved J11 5.47 mm to (140.6, 100.7)
- moved D1 5.40 mm to (140.6, 94.9)
- moved J10 4.94 mm to (140.9, 87.6)
- moved J1 4.20 mm to (135.4, 100.8)
- moved D8 4.10 mm to (135.4, 94.9)
- moved J12 4.04 mm to (135.9, 87.6)
- moved C22 3.71 mm to (120.5, 124.3)
- moved C20 3.62 mm to (118.9, 124.3)
- moved Q1 1.95 mm to (131.5, 91.0)
- moved U1 1.60 mm to (121.7, 88.1)
- moved L1 1.55 mm to (104.5, 97.0)
- moved J8 0.93 mm to (115.6, 80.3), turned to 90 degrees
- moved J2 0.91 mm to (115.6, 87.2)
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- renumbered SW4 to RESET
Connections:
- R18 pad 2: Net-(R17-Pad1) -> Net-(C35-Pad2)
Routing:
- net Net-(R21-Pad2): track 0.00 -> 13.8 mm
- net Net-(J2-Pad1): track 12.0 -> 0.00 mm
- net Net-(R20-Pad2): track 0.00 -> 11.7 mm
- net Net-(C35-Pad2): track 34.9 -> 23.6 mm, vias 2 -> 0
- net 3v3: track 173.7 -> 184.7 mm, vias 16 -> 18
- net 12V: track 49.8 -> 44.1 mm
- net XTAL_N: track 10.3 -> 15.3 mm
- net Net-(D8-Pad2): track 4.90 -> 0.00 mm
- net Net-(D1-Pad2): track 4.70 -> 0.00 mm
- net Earth: track 33.7 -> 38.0 mm, vias 55 -> 72
- net VDD_ANA: track 54.3 -> 58.4 mm
- net Net-(C20-Pad2): track 5.95 -> 9.52 mm
- net Net-(R22-Pad2): track 0.00 -> 3.39 mm
- net (no net): track 0.00 -> 1.92 mm
- net Net-(R17-Pad1): track 12.4 -> 11.4 mm
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Other:
- board size 60.3 x 55.7 mm -> 54.5 x 55.7 mm

Commit message: BAU
Changed lines of the file:
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@@
     (links 372)
     (no_connects 0)
-    (area 89.024822 76.524999 143.675023 132.325001)
+    (area 88.694999 74.395 144.653 134.505)
     (thickness 1.4)
     (drawings 23)
@@
     (tags "capacitor 0603")
     (attr smd)
-    (fp_text reference C12 (at 0 1.7 180) (layer F.SilkS)
+    (fp_text reference C12 (at 1.85 1.4 180) (layer F.SilkS)
       (effects (font (size 1 1) (thickness 0.15)))
     )
@@
     (tags "resistor 0603")
     (attr smd)
-    (fp_text reference R7 (at 2.35 0.9 90) (layer F.SilkS)
+    (fp_text reference R7 (at 1.85 1.3 90) (layer F.SilkS)
       (effects (font (size 1 1) (thickness 0.15)))
     )
@@
     (polygon
       (pts
-        (xy 108.2 82.8) (xy 133.398366 82.8) (xy 133.4 90.6) (xy 143.6 90.531752) (xy 143.6 76.6)
+        (xy 108.2 82.8) (xy 133.398366 82.8) (xy 133.4 90.6) (xy 143.6 90.6) (xy 143.6 76.6)
         (xy 108.2 76.6)
       )
