File: Schamatic/Motor/motor.kicad_pcb (KiCad board)
At the start: 2 copper layers, 36.2 x 24 mm, 45 parts, among them J1 CONN_02X05, J11 V, J12 U, J13 W, J2 SPI, J3 RS485, J4 GND, J5 CAP+, J6 12, J7 GND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

Commit message: fixes to the boards
Parts:
- removed J5: CAP+, Pin_Headers:Pin_Header_Straight_1x01_Pitch2.54mm
- removed J8: CAP-, Pin_Headers:Pin_Header_Straight_1x01_Pitch2.54mm
- added D6: 47v, Diodes_SMD:D_SOD-123F, F.Cu at (164.1, 109.1)
- C3: value 22uF -> 10uF; footprint Capacitors_SMD:C_0805 -> Capacitors_SMD:C_1206
- D1, D4: footprint Diodes_SMD:D_0603 -> Diodes_SMD:D_SOD-323F
- Y1: footprint Dizzy:OSC_CSTCE16M0V53-R0 -> Dizzy:Oscillator
- moved Y1 2.64 mm to (160.0, 99.0)
- moved C3 2.51 mm to (164.0, 107.0)
- moved C2 0.40 mm to (157.7, 97.5)
Connections:
- J2 pad 1: MOSI -> Earth
- J2 pad 2: MISO -> CS
- J2 pad 4: CS -> MOSI
- J2 pad 5: Earth -> MISO
- U1 pad 13: Net-(SW1-Pad1) -> Net-(ID1-Pad1)
- U1 pad 14: Net-(SW2-Pad1) -> Net-(CALIB1-Pad1)
Routing:
- net Net-(CALIB1-Pad1): track 0.00 -> 4.94 mm, vias 0 -> 1
- net Net-(SW2-Pad1): track 16.2 -> 11.3 mm, vias 2 -> 1
- net Earth: track 70.4 -> 66.5 mm, vias 12 -> 14
- net Net-(ID1-Pad1): track 0.00 -> 2.80 mm, vias 0 -> 1
- net Net-(SW1-Pad1): track 12.9 -> 10.1 mm, vias 2 -> 1
- net MISO: track 14.7 -> 13.2 mm
- net MOSI: track 15.5 -> 14.5 mm
- net Net-(C2-Pad2): track 7.81 -> 8.62 mm
- net CS: track 12.3 -> 12.9 mm
- net Net-(D3-Pad2): track 19.6 -> 19.8 mm, vias 2 -> 3
- net VM: track 16.6 -> 16.4 mm, vias 1 -> 4
