File: Schamatic/PiHat/PiHat.kicad_pcb (KiCad board)
At the start: 2 copper layers, 65 x 29.9 mm, 44 parts, among them J1 +45V, J10 GND, J11 GND, J12 SW1, J13 SW2, J14 MOUNT, J15 MOUNT, J16 MOUNT, J17 MOUNT, J2 +45V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

Commit message: Pi hat more or less ready
Parts:
- added C12: 0.1uF, Capacitors_SMD:C_0603, F.Cu at (132.6, 55.8)
- added J18: CONN_02X05, Pin_Headers:Pin_Header_Straight_2x05_Pitch1.27mm, F.Cu at (124.2, 49.9)
- added J19: ADCV, Dizzy:SOLDER-SWITCH, F.Cu at (119.2, 60.5)
- added J20: ADCI, Dizzy:SOLDER-SWITCH, F.Cu at (119.1, 59.0)
- added J21: RX, Dizzy:SOLDER-SWITCH, F.Cu at (119.1, 54.1)
- added J22: DE, Dizzy:SOLDER-SWITCH, F.Cu at (119.1, 55.8)
- added J23: TX, Dizzy:SOLDER-SWITCH, F.Cu at (119.1, 57.4)
- added J24: SDA, Dizzy:SOLDER-SWITCH, F.Cu at (119.1, 63.8)
- added J25: SCL, Dizzy:SOLDER-SWITCH, F.Cu at (119.1, 62.2)
- added J26: CONN_01X02, Pin_Headers:Pin_Header_Straight_2x01_Pitch2.54mm, F.Cu at (138.0, 48.2)
- added J27: CONN_01X02, Pin_Headers:Pin_Header_Straight_2x01_Pitch2.54mm, F.Cu at (134.1, 48.2)
- added REF**: VIA-0.4, Dizzy:VIA-0.4, F.Cu at (119.4, 51.4)
- added REF**: VIA-0.4, Dizzy:VIA-0.4, F.Cu at (121.0, 52.1)
- added REF**: VIA-0.4, Dizzy:VIA-0.4, F.Cu at (120.0, 54.2)
- added REF**: VIA-0.4, Dizzy:VIA-0.4, F.Cu at (106.3, 51.3)
- added REF**: VIA-0.4, Dizzy:VIA-0.4, F.Cu at (131.9, 65.2)
- added REF**: VIA-0.4, Dizzy:VIA-0.4, F.Cu at (136.1, 52.4)
- added REF**: VIA-0.4, Dizzy:VIA-0.4, F.Cu at (95.9, 58.8)
- added REF**: VIA-0.4, Dizzy:VIA-0.4, F.Cu at (110.5, 60.8)
- added U7: STM32F031G4U6, Dizzy:STM32F031G4U6, F.Cu at (128.4, 55.8)
- added Y1: Resonator_Small, Dizzy:OSC_CSTCE16M0V53-R0, F.Cu at (124.2, 55.0)
- J7: moved to F.Cu
- moved J7 48.1 mm to (84.0, 43.6)
- moved R7 18.5 mm to (123.0, 64.3)
- moved R8 11.8 mm to (123.0, 62.5)
- moved C10 10.2 mm to (138.1, 56.1)
- moved U6 10.2 mm to (137.2, 59.1)
- moved U5 8.32 mm to (130.4, 62.8)
- moved C11 6.47 mm to (130.3, 66.4)
- moved C4 0.20 mm to (97.4, 52.3)
- moved C3 0.10 mm to (97.3, 47.0)
Connections:
- C2 pad 1: ADC_V -> ADCV
- C9 pad 1: ADC_I -> ADCI
- J7 pad 10: RX -> PI_RX
- J7 pad 12: DE -> PI_DE
- J7 pad 19: Net-(J7-Pad19) -> MOSI
- J7 pad 21: Net-(J7-Pad21) -> MISO
- J7 pad 23: Net-(J7-Pad23) -> SCK
- J7 pad 29: Net-(J7-Pad29) -> WRDY
- J7 pad 3: SDA -> PI_SDA
- J7 pad 31: Net-(J7-Pad31) -> RRDY
- J7 pad 5: SCL -> PI_SCL
- J7 pad 8: TX -> PI_TX
- R3 pad 2: ADC_V -> ADCV
- R4 pad 1: ADC_V -> ADCV
- R5 pad 2: ADC_I -> ADCI
- R6 pad 1: ADC_I -> ADCI
- U4 pad 1: ADC_V -> PI_ADCV
- U4 pad 7: ADC_I -> PI_ADCI
Routing:
- net 3.3V: track 28.8 -> 184.5 mm, vias 0 -> 8
- net PI_SDA: track 0.00 -> 53.1 mm, vias 0 -> 1
- net SCL: track 0.00 -> 52.9 mm, vias 0 -> 2
- net SDA: track 0.00 -> 51.6 mm, vias 0 -> 2
- net PI_SCL: track 0.00 -> 49.0 mm, vias 0 -> 1
- net ADCV: track 0.00 -> 44.2 mm, vias 0 -> 2
- net ADCI: track 0.00 -> 44.1 mm, vias 0 -> 2
- net PI_TX: track 0.00 -> 43.9 mm, vias 0 -> 1
- net PI_ADCI: track 0.00 -> 38.9 mm, vias 0 -> 2
- net PI_ADCV: track 0.00 -> 37.7 mm, vias 0 -> 2
- net PI_RX: track 0.00 -> 37.5 mm, vias 0 -> 1
- net PI_DE: track 0.00 -> 37.0 mm, vias 0 -> 1
- net Earth: track 25.7 -> 58.2 mm, vias 16 -> 15
- net MOSI: track 0.00 -> 32.0 mm, vias 0 -> 1
- net MISO: track 0.00 -> 30.9 mm, vias 0 -> 1
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- added copper zone on F.Cu, net Earth
- added copper zone on F.Cu, net Net-(D1-Pad1)
- added copper zone on F.Cu, net Net-(D1-Pad2)
- added copper zone on F.Cu, net Net-(D2-Pad2)
- added copper zone on F.Cu, net Net-(J8-Pad1)
- added copper zone on F.Cu, net VIN

Commit message: accumulated changes
Parts:
- added REF**: VIA-0.4, Dizzy:VIA-0.4, F.Cu at (135.9, 55.3)
Connections:
- REF** pad 1: (no net) -> Earth

Commit message: fixes to the boards
Parts:
- removed the REF** at (95.9, 58.8)
- removed the REF** at (110.5, 60.8)
- added C13: 10uF, Capacitors_SMD:C_1206, F.Cu at (95.7, 60.1)
- added D3: 47V, Diodes_SMD:D_SOD-123F, F.Cu at (95.7, 57.6)
- added REF**: VIA-0.4, Dizzy:VIA-0.4, F.Cu at (125.7, 65.2)
- C6, C8: footprint Capacitors_SMD:C_0805 -> Capacitors_SMD:C_1206
- D2: footprint Diodes_SMD:D_SMA -> Diodes_SMD:D_SOD-323F
- L1, L2: footprint Inductors_SMD:L_1812 -> Dizzy:Inductor-1812
- Y1: footprint Dizzy:OSC_CSTCE16M0V53-R0 -> Dizzy:Oscillator
- moved D2 9.86 mm to (93.1, 62.3)
- moved J10 4.80 mm to (110.6, 60.9)
- moved J11 4.80 mm to (106.1, 60.8)
- moved J8 4.80 mm to (106.2, 66.1)
- moved J9 4.80 mm to (110.7, 66.2)
- moved U1 4.80 mm to (100.7, 63.7)
- moved C11 4.57 mm to (126.3, 64.2), turned to 180 degrees
- moved Y1 2.62 mm to (126.5, 53.8)
- moved L1 2.04 mm to (104.3, 48.6)
- moved L2 2.04 mm to (104.3, 53.8)
- moved C6 0.60 mm to (111.3, 49.2)
- moved C8 0.60 mm to (111.3, 54.7)
Connections:
- D2 pad 1: Net-(D1-Pad1) -> VIN
- J13 pad 1: VIN -> Net-(D2-Pad2)
- J2 pad 1: Net-(D2-Pad2) -> Net-(D1-Pad1)
- J7 pad 33: Net-(J7-Pad33) -> GPIO13
- J7 pad 35: Net-(J7-Pad35) -> GPIO19
- J7 pad 37: Net-(J7-Pad37) -> GPIO26
- R3 pad 1: VIN -> Net-(D2-Pad2)
- U1 pad 5: VIN -> Net-(D2-Pad2)
- U7 pad 23: Net-(U7-Pad23) -> GPIO26
- U7 pad 24: Net-(U7-Pad24) -> GPIO19
- U7 pad 25: Net-(U7-Pad25) -> GPIO13
Routing:
- net Net-(D2-Pad2): track 3.30 -> 30.7 mm
- net GPIO26: track 0.00 -> 19.5 mm, vias 0 -> 1
- net VIN: track 52.3 -> 33.4 mm
- net GPIO19: track 0.00 -> 16.9 mm, vias 0 -> 1
- net GPIO13: track 0.00 -> 15.6 mm, vias 0 -> 1
- net Net-(D1-Pad1): track 12.2 -> 19.5 mm
- net Net-(R5-Pad1): track 18.5 -> 23.6 mm
- net Net-(J8-Pad1): track 8.54 -> 4.54 mm
- net 5V: track 53.2 -> 50.1 mm
- net Net-(L1-Pad1): track 5.61 -> 3.74 mm
- net Earth: track 58.2 -> 59.8 mm
- net SCL: track 52.9 -> 54.2 mm
- net PI_ADCV: track 37.7 -> 38.3 mm
- net WRDY: track 14.6 -> 15.2 mm
- net SDA: track 51.6 -> 52.1 mm
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- removed copper zone on F.Cu, net Net-(D2-Pad2)
Other:
- outline, holes or cut-outs redrawn
- board text added: "DizzyRobot"

Commit message: removing old cc3220 mainboard
Routing:
- added copper zone on F.Cu, net Net-(D2-Pad2)
Changed lines of the file:
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@@
   (general
     (links 178)
-    (no_connects 3)
+    (no_connects 0)
     (area 75.424999 37.406666 141.335 70.205)
     (thickness 1.6)
@@
     (user_trace_width 0.5)
     (trace_clearance 0.13)
-    (zone_clearance 0.2)
+    (zone_clearance 0.3)
     (zone_45_only no)
     (trace_min 0.1)
@@
     )
   )
-  (zone (net 32) (net_name VIN) (layer F.Cu) (hatch edge 0.508)
+  (zone (net 10) (net_name "Net-(D2-Pad2)") (layer F.Cu) (hatch edge 0.508)
     (priority 1)
     (connect_pads yes (clearance 0.3))

Commit message: saving
Parts:
- removed C1: 0.1uF, Capacitors_SMD:C_0603
- removed REF** (x8): VIA-0.4, Dizzy:VIA-0.4
- removed U4: MCP3426, Dizzy:8-DFN-2x3
- added D4: D_Small, Diodes_SMD:D_SOD-323, F.Cu at (112.6, 57.9)
- added D5: D_Small, Diodes_SMD:D_SOD-323, F.Cu at (112.8, 51.1)
- added D6: LED_Small, LEDs:LED_0603, F.Cu at (116.5, 67.9)
- added D7: LED_Small, LEDs:LED_0603, F.Cu at (120.2, 67.9)
- added R1: 22k, Resistors_SMD:R_0603, F.Cu at (97.5, 54.5)
- added R10: 370, Resistors_SMD:R_0603, F.Cu at (120.0, 66.5)
- added R2: 22k, Resistors_SMD:R_0603, F.Cu at (97.5, 47.8)
- added R9: 370, Resistors_SMD:R_0603, F.Cu at (116.3, 66.4)
- C13: value 10uF -> 1uF
- C3, C4: value 1uF -> 22nF
- C5: value 3300pF -> 220nF
- C6: value 22uF -> 220nF; footprint Capacitors_SMD:C_1206 -> Capacitors_SMD:C_0603
- C7: value 3300pF -> 100uF; footprint Capacitors_SMD:C_0603 -> Capacitors_SMD:C_1206
- C8: value 10uF -> 100uF
- J14, J15, J16, J17: footprint Connectors:1pin -> Dizzy:1pin
- J19: value ADCV -> SDA; footprint Dizzy:SOLDER-SWITCH -> Dizzy:1pin
- J20: value ADCI -> SCL; footprint Dizzy:SOLDER-SWITCH -> Dizzy:1pin
- J21: value RX -> ADCI; footprint Dizzy:SOLDER-SWITCH -> Dizzy:1pin
- J22: value DE -> ADCV; footprint Dizzy:SOLDER-SWITCH -> Dizzy:1pin
- J23: value TX -> DE; footprint Dizzy:SOLDER-SWITCH -> Dizzy:1pin
- J24: value SDA -> TX; footprint Dizzy:SOLDER-SWITCH -> Dizzy:1pin
- J25: value SCL -> RX; footprint Dizzy:SOLDER-SWITCH -> Dizzy:1pin
- L1: value 15uH -> 47uH
- L2: value 22uH -> 47uH
- U2: value MAX17502-3.3V -> IFX91041 - 5V; footprint Housings_DFN_QFN:DFN-10-1EP_2x3mm_Pitch0.5mm -> Housings_SOIC:HTSOP-8-1EP_3.9x4.9mm_Pitch1.27mm_ThermalVias
- U3: value MAX17502-5V -> IFX91041 - 3.3V; footprint Housings_DFN_QFN:DFN-10-1EP_2x3mm_Pitch0.5mm -> Housings_SOIC:HTSOP-8-1EP_3.9x4.9mm_Pitch1.27mm_ThermalVias
- moved J23 18.8 mm to (137.3, 62.0)
- moved J25 17.4 mm to (135.3, 56.0)
- moved C7 16.5 mm to (113.1, 54.3), turned to 270 degrees
- moved J24 16.0 mm to (135.0, 62.1)
- moved C5 15.4 mm to (109.3, 57.9), turned to 0 degrees
- moved L1 9.26 mm to (110.0, 55.9), turned to 90 degrees
- moved L2 7.20 mm to (110.0, 49.4), turned to 90 degrees
- moved C8 7.13 mm to (113.1, 47.8)
- moved U3 6.99 mm to (102.8, 48.2), turned to 0 degrees
- moved U2 6.22 mm to (102.9, 54.8), turned to 0 degrees
- moved C3 6.00 mm to (97.5, 53.0), turned to 0 degrees
- moved C4 5.90 mm to (97.4, 46.4), turned to 0 degrees
- moved J20 4.82 mm to (123.9, 58.5)
- moved R7 3.77 mm to (126.2, 62.3)
- moved R8 3.77 mm to (126.2, 60.5)
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Connections:
- net RRDY renamed RECVRDY
- net WRDY renamed RESPRDY
- C5 pad 2: Earth -> Net-(C5-Pad2)
- C6 pad 1: 3.3V -> Net-(C6-Pad1)
- C6 pad 2: Earth -> Net-(C6-Pad2)
- C7 pad 1: Net-(C7-Pad1) -> 5V
- C8 pad 1: 5V -> 3.3V
- J18 pad 6: Net-(J18-Pad6) -> (no net)
- J18 pad 7: Net-(J18-Pad7) -> (no net)
- J18 pad 8: Net-(J18-Pad8) -> (no net)
- J19 pad 1: PI_ADCV -> SDA
- J20 pad 1: PI_ADCI -> SCL
- J21 pad 1: PI_RX -> ADCI
- J22 pad 1: PI_DE -> ADCV
- J23 pad 1: PI_TX -> DE
- J24 pad 1: PI_SDA -> TX
- J25 pad 1: PI_SCL -> RX
- J7 pad 10: PI_RX -> (no net)
- J7 pad 11: Net-(J7-Pad11) -> (no net)
- J7 pad 12: PI_DE -> (no net)
- J7 pad 13: Net-(J7-Pad13) -> (no net)
- J7 pad 15: Net-(J7-Pad15) -> (no net)
- J7 pad 16: Net-(J7-Pad16) -> (no net)
- J7 pad 18: Net-(J7-Pad18) -> (no net)
- J7 pad 2: 5V -> (no net)
- J7 pad 22: Net-(J7-Pad22) -> (no net)
- J7 pad 24: Net-(J7-Pad24) -> CS
- J7 pad 26: Net-(J7-Pad26) -> (no net)
- J7 pad 27: Net-(J7-Pad27) -> (no net)
- J7 pad 28: Net-(J7-Pad28) -> (no net)
- J7 pad 3: PI_SDA -> (no net)
- J7 pad 32: Net-(J7-Pad32) -> (no net)
- J7 pad 36: Net-(J7-Pad36) -> (no net)
- J7 pad 38: Net-(J7-Pad38) -> (no net)
- J7 pad 4: 5V -> (no net)
- J7 pad 40: Net-(J7-Pad40) -> (no net)
- J7 pad 5: PI_SCL -> (no net)
- J7 pad 7: Net-(J7-Pad7) -> (no net)
- J7 pad 8: PI_TX -> (no net)
- L1 pad 1: Net-(L1-Pad1) -> Net-(C5-Pad2)
- L1 pad 2: 3.3V -> 5V
- L2 pad 1: Net-(L2-Pad1) -> Net-(C6-Pad2)
- L2 pad 2: 5V -> 3.3V
- U2 pad 2: VIN -> Earth
- U2 pad 3: VIN -> Net-(R1-Pad1)
- U2 pad 4: Net-(C3-Pad1) -> 5V
- U2 pad 5: 3.3V -> Net-(C5-Pad1)
- U2 pad 6: Net-(C5-Pad1) -> Net-(C5-Pad2)
- U2 pad 7: Net-(U2-Pad7) -> VIN
- U2 pad 8: Net-(U2-Pad8) -> VIN
- U3 pad 2: VIN -> Earth
- U3 pad 3: VIN -> Net-(R2-Pad1)
- U3 pad 4: Net-(C4-Pad1) -> 3.3V
- U3 pad 5: 5V -> Net-(C6-Pad1)
- U3 pad 6: Net-(C7-Pad1) -> Net-(C6-Pad2)
- U3 pad 7: Net-(U3-Pad7) -> VIN
- U3 pad 8: Net-(U3-Pad8) -> VIN
- U5 pad 14: Net-(U5-Pad14) -> (no net)
- U5 pad 6: Net-(U5-Pad6) -> (no net)
- U5 pad 7: Net-(U5-Pad7) -> (no net)
- U7 pad 10: MCU_ADCV -> CS
- U7 pad 14: Net-(U7-Pad14) -> ADCV
- U7 pad 18: Net-(U7-Pad18) -> (no net)
- U7 pad 19: MCU_SCL -> SCL
- U7 pad 20: MCU_SDA -> SDA
- U7 pad 6: MCU_ADCI -> ADCI
- U7 pad 7: MCU_DE -> DE
- U7 pad 8: MCU_TX -> TX
- U7 pad 9: MCU_RX -> RX
Routing:
- net PI_SDA: track 52.6 -> 0.00 mm, vias 1 -> 0
- net PI_SCL: track 48.7 -> 0.00 mm, vias 1 -> 0
- net PI_TX: track 43.9 -> 0.00 mm, vias 1 -> 0
- net PI_ADCI: track 39.5 -> 0.00 mm, vias 2 -> 0
- net PI_ADCV: track 38.3 -> 0.00 mm, vias 2 -> 0
- net SCL: track 54.2 -> 16.6 mm
- net PI_RX: track 37.6 -> 0.00 mm, vias 1 -> 0
- net PI_DE: track 37.2 -> 0.00 mm, vias 1 -> 0
- net SDA: track 52.1 -> 21.3 mm
- net 5V: track 50.1 -> 19.7 mm, vias 6 -> 2
- net CS: track 0.00 -> 29.3 mm, vias 0 -> 1
- net 3.3V: track 184.6 -> 155.9 mm, vias 7 -> 2
- net RESPRDY: track 15.2 -> 41.1 mm, vias 1 -> 2
- net RECVRDY: track 14.6 -> 37.1 mm, vias 1 -> 2
- net MCU_SDA: track 20.6 -> 0.00 mm, vias 2 -> 0
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- removed copper zone on F.Cu, net VIN

Commit message: current changes
Routing:
- net RESPRDY: track 41.1 -> 39.6 mm
- net Earth: track 51.2 -> 50.4 mm
Changed lines of the file:
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@@
     (links 187)
     (no_connects 0)
-    (area 75.424999 38.724999 140.575001 68.775001)
+    (area 75.424999 37.406666 141.335 70.605)
     (thickness 1.6)
     (drawings 9)
-    (tracks 560)
+    (tracks 556)
     (zones 0)
     (modules 65)
@@
     (mod_text_size 1 1)
     (mod_text_width 0.15)
-    (pad_size 1 1)
-    (pad_drill 0.7)
+    (pad_size 4 4)
+    (pad_drill 3.5)
     (pad_to_mask_clearance 0.2)
     (aux_axis_origin 0 0)
@@
       (effects (font (size 1 1) (thickness 0.15)))
     )
-    (pad 1 thru_hole circle (at 0 0) (size 3.5 3.5) (drill 2.2) (layers *.Cu *.Mask)
+    (pad 1 thru_hole circle (at 0 0) (size 4 4) (drill 3.5) (layers *.Cu *.Mask)
       (net 1 Earth) (zone_connect 2))
   )
@@
       (effects (font (size 1 1) (thickness 0.15)))
     )
-    (pad 1 thru_hole circle (at 0 0) (size 3.5 3.5) (drill 2.2) (layers *.Cu *.Mask)
+    (pad 1 thru_hole circle (at 0 0) (size 4 4) (drill 3.5) (layers *.Cu *.Mask)
       (net 1 Earth) (zone_connect 2))
   )
@@
       (effects (font (size 1 1) (thickness 0.15)))
     )
-    (pad 1 thru_hole circle (at 0 0) (size 3.5 3.5) (drill 2.2) (layers *.Cu *.Mask)
+    (pad 1 thru_hole circle (at 0 0) (size 4 4) (drill 3.5) (layers *.Cu *.Mask)
       (net 1 Earth) (zone_connect 2))
   )
@@
       (effects (font (size 1 1) (thickness 0.15)))
     )
-    (pad 1 thru_hole circle (at 0 0) (size 3.5 3.5) (drill 2.2) (layers *.Cu *.Mask)
+    (pad 1 thru_hole circle (at 0 0) (size 4 4) (drill 3.5) (layers *.Cu *.Mask)
       (net 1 Earth) (zone_connect 2))
   )
@@
   (segment (start 131.8224 61.350398) (end 131.8224 61.4324) (width 0.25) (layer F.Cu) (net 1))
   (via (at 124.2 55.05) (size 0.4) (drill 0.25) (layers F.Cu B.Cu) (net 1))
-  (segment (start 137.6 64.7) (end 137 65.3) (width 0.25) (layer F.Cu) (net 1))
   (segment (start 131.8224 63.7906) (end 131.3398 63.7906) (width 0.25) (layer F.Cu) (net 1))
   (segment (start 131.3398 63.7906) (end 130.908 64.2224) (width 0.25) (layer F.Cu) (net 1))
@@
   (segment (start 105.5 50.655) (end 105.5 50.105) (width 0.25) (layer F.Cu) (net 37))
   (segment (start 105.945 51.1) (end 105.5 50.655) (width 0.25) (layer F.Cu) (net 37))
+  (segment (start 127.1 53.1) (end 127.1 54.067711) (width 0.13) (layer B.Cu) (net 38))
+  (segment (start 127.1 54.067711) (end 130.8 57.767711) (width 0.13) (layer B.Cu) (net 38))
+  (segment (start 130.8 57.767711) (end 130.8 58.7) (width 0.13) (layer B.Cu) (net 38))
+  (segment (start 130.8 58.7) (end 129.860011 59.639989) (width 0.13) (layer B.Cu) (net 38))
+  (segment (start 129.860011 59.639989) (end 126.1923 59.639989) (width 0.13) (layer B.Cu) (net 38))
+  (segment (start 126.1923 59.639989) (end 117.932289 67.9) (width 0.13) (layer B.Cu) (net 38))
+  (segment (start 117.932289 67.9) (end 117.3 67.9) (width 0.13) (layer B.Cu) (net 38))
   (segment (start 122.160011 50.830855) (end 123.269145 51.939989) (width 0.13) (layer B.Cu) (net 38))
   (segment (start 122.160011 46.240011) (end 122.160011 50.830855) (width 0.13) (layer B.Cu) (net 38))
@@
   (segment (start 126.817158 53.1) (end 127.1 53.1) (width 0.13) (layer B.Cu) (net 38))
   (segment (start 123.269145 51.939989) (end 124.2077 51.939989) (width 0.13) (layer B.Cu) (net 38))
-  (segment (start 130.8 58.7) (end 129.860011 59.639989) (width 0.13) (layer B.Cu) (net 38))
-  (segment (start 129.860011 59.639989) (end 126.1923 59.639989) (width 0.13) (layer B.Cu) (net 38))
-  (segment (start 127.1 53.1) (end 127.1 54.067711) (width 0.13) (layer B.Cu) (net 38))
   (via (at 117.3 67.9) (size 0.4) (drill 0.25) (layers F.Cu B.Cu) (net 38))
-  (segment (start 127.1 54.067711) (end 130.8 57.767711) (width 0.13) (layer B.Cu) (net 38))
-  (segment (start 124.139989 61.6923) (end 124.139989 64.260011) (width 0.13) (layer B.Cu) (net 38))
-  (segment (start 120.5 67.9) (end 117.3 67.9) (width 0.13) (layer B.Cu) (net 38))
-  (segment (start 130.8 57.767711) (end 130.8 58.7) (width 0.13) (layer B.Cu) (net 38))
-  (segment (start 126.1923 59.639989) (end 124.139989 61.6923) (width 0.13) (layer B.Cu) (net 38))
-  (segment (start 124.139989 64.260011) (end 120.5 67.9) (width 0.13) (layer B.Cu) (net 38))
   (segment (start 127.299999 53.299999) (end 127.1 53.1) (width 0.13) (layer F.Cu) (net 38))
   (segment (start 127.425 53.925) (end 127.425 53.425) (width 0.13) (layer F.Cu) (net 38))
@@
   (segment (start 115.7 67.9) (end 115.7 66.5) (width 0.13) (layer F.Cu) (net 39))
   (segment (start 115.7 66.5) (end 115.6 66.4) (width 0.13) (layer F.Cu) (net 39))
+  (segment (start 127.800004 53.1) (end 127.800004 54.200004) (width 0.13) (layer B.Cu) (net 40))
+  (segment (start 127.800004 54.200004) (end 131.1 57.5) (width 0.13) (layer B.Cu) (net 40))
+  (segment (start 131.1 57.5) (end 131.1 58.9) (width 0.13) (layer B.Cu) (net 40))
+  (segment (start 131.1 58.9) (end 130.1 59.9) (width 0.13) (layer B.Cu) (net 40))
+  (segment (start 121.224535 64.975465) (end 121.224535 67.734094) (width 0.13) (layer B.Cu) (net 40))
+  (segment (start 130.1 59.9) (end 126.3 59.9) (width 0.13) (layer B.Cu) (net 40))
+  (segment (start 126.3 59.9) (end 121.224535 64.975465) (width 0.13) (layer B.Cu) (net 40))
+  (segment (start 121.224535 67.734094) (end 121.024536 67.934093) (width 0.13) (layer B.Cu) (net 40))
   (segment (start 122.420022 50.723155) (end 123.376845 51.679978) (width 0.13) (layer B.Cu) (net 40))
   (segment (start 124.315455 51.680033) (end 126.380037 51.680033) (width 0.13) (layer B.Cu) (net 40))
@@
   (segment (start 123.376845 51.679978) (end 124.3154 51.679978) (width 0.13) (layer B.Cu) (net 40))
   (segment (start 122.1 43.64) (end 122.1 44.842081) (width 0.13) (layer B.Cu) (net 40))
-  (segment (start 121.224535 67.734094) (end 121.024536 67.934093) (width 0.13) (layer B.Cu) (net 40))
-  (segment (start 124.4 64.558629) (end 121.224535 67.734094) (width 0.13) (layer B.Cu) (net 40))
-  (segment (start 131.1 58.9) (end 130.1 59.9) (width 0.13) (layer B.Cu) (net 40))
-  (segment (start 131.1 57.5) (end 131.1 58.9) (width 0.13) (layer B.Cu) (net 40))
-  (segment (start 127.800004 53.1) (end 127.800004 54.200004) (width 0.13) (layer B.Cu) (net 40))
-  (segment (start 127.800004 54.200004) (end 131.1 57.5) (width 0.13) (layer B.Cu) (net 40))
   (via (at 121.024536 67.934093) (size 0.4) (drill 0.25) (layers F.Cu B.Cu) (net 40))
-  (segment (start 124.4 61.8) (end 124.4 64.558629) (width 0.13) (layer B.Cu) (net 40))
-  (segment (start 130.1 59.9) (end 126.3 59.9) (width 0.13) (layer B.Cu) (net 40))
-  (segment (start 126.3 59.9) (end 124.4 61.8) (width 0.13) (layer B.Cu) (net 40))
   (segment (start 127.925 53.925) (end 127.925 53.224996) (width 0.13) (layer F.Cu) (net 40))
   (segment (start 127.925 53.224996) (end 127.800004 53.1) (width 0.13) (layer F.Cu) (net 40))
