File: Electronics/Motor-2/Schematic-Board/motor.kicad_pcb (KiCad board)
At the start: 2 copper layers, 45 x 45 mm, 72 parts, among them J1 CONN_02X05, J11 V, J12 U, J13 W, J2 RS485, J3 RS485, J4 CONN_01X06, J6 12, J9 GND, Q1 PSMN3R3-40YS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

Commit message: current changes
Parts:
- removed CALIB1: CALIB, Resistors_SMD:R_1206
- removed the REF** at (78.1, 63.9)
- removed the REF** at (76.4, 65.6)
- added J5: JTAG, Connectors:Tag-Connect_TC2050-IDC-NL, B.Cu at (80.6, 57.8)
- added REF**: VIA-0.4, Dizzy:VIA-0.4, F.Cu at (81.5, 65.5)
- added REF**: VIA-0.4, Dizzy:VIA-0.4, F.Cu at (78.5, 63.6)
- added REF**: VIA-0.4, Dizzy:VIA-0.4, F.Cu at (80.9, 56.0)
- added REF**: VIA-0.4, Dizzy:VIA-0.4, F.Cu at (79.1, 55.7)
- moved J1 7.38 mm to (79.1, 65.5), turned to 270 degrees
Connections:
- U1 pad 14: Net-(CALIB1-Pad1) -> (no net)
Routing:
- net Net-(CALIB1-Pad1): track 36.0 -> 0.00 mm, vias 4 -> 0
- net NRST: track 14.7 -> 41.6 mm
- net SWDCLK: track 26.4 -> 36.1 mm, vias 3 -> 4
- net SWDIO: track 27.7 -> 36.9 mm, vias 3 -> 4
- net (no net): track 0.00 -> 4.52 mm
- net Earth: track 12.3 -> 9.39 mm, vias 1 -> 0
- net Net-(ID1-Pad1): track 37.1 -> 39.7 mm
- net +3V3: track 97.7 -> 98.6 mm
Other:
- board text removed: "calib"
