File: Electronics/Mainboard/Schematic/PiConn/PiConn.kicad_pcb (KiCad board)
At the start: 2 copper layers, 27.1 x 65.7 mm, 10 parts, among them J1 CONN_02X10, J2 CONN_02X20, J3 CONN_01X02, J4 CONN_01X02, J5 CONN_01X02

Commit message: new mainboard
Parts:
- moved J2 48.1 mm to (166.7, 106.9), turned to 0 degrees
Routing:
- net 12V: track 0.00 -> 55.0 mm
- net 5V: track 0.00 -> 50.8 mm
- net ~PWR_KILL: track 0.00 -> 42.4 mm
- net PWR_INT: track 0.00 -> 13.8 mm
- net Earth: track 0.00 -> 12.8 mm, vias 0 -> 3
- net CS: track 0.00 -> 10.2 mm
- net RESPRDY: track 0.00 -> 8.61 mm
- net RECVRDY: track 0.00 -> 8.61 mm
- net SCK: track 0.00 -> 7.56 mm
- net MOSI: track 0.00 -> 7.56 mm
- net MISO: track 0.00 -> 7.56 mm
- net 3.3V: track 0.00 -> 4.25 mm
- added copper zone on F.Cu, net 3.3V
