File: Electronics/Mainboard/Schematic/Mainboard.kicad_pcb (KiCad board)
At the start: 4 copper layers, 45 x 140 mm, 77 parts, among them J1 CONN_01X02, J10 CONN_01X04, J11 M1, J12 M2, J13 M3, J14 M4, J15 CONN_01X01, J16 CONN_01X01, J17 CONN_01X01, J18 CONN_01X01, J2 CONN_01X02, J21 CONN_01X01, J22 CONN_01X01, J23 CONN_01X01, J24 CONN_01X01, J25 CONN_01X01, J26 CONN_01X01, J27 CONN_01X01, J3 CONN_01X02, J4 CONN_01X02, J5 CONN_01X02, J6 CONN_02X05, J7 CONN_02X10, J8 CONN_01X02, J9 CONN_01X02, Q1 BSS123W, Q2 SQJ459EP, U1 LM2678-3.3V, U10 LTC2954-1, U2 LM2678-12V, U3 ZXTR2012Z, U6 ACS781, U7 LSM6DS33, U8 STM32F031K6U6, U9 LTC2876, Y1 Resonator_Small

Commit message: changes changes
Routing:
- net Earth: track 128.1 -> 97.0 mm
- net 3.3V: track 45.2 -> 37.2 mm
Changed lines of the file:
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@@
     (thickness 1.6)
     (drawings 11)
-    (tracks 652)
+    (tracks 628)
     (zones 0)
     (modules 77)
@@
   (gr_line (start 95 32) (end 95 168) (layer Edge.Cuts) (width 0.15))
   (gr_line (start 52 30) (end 93 30) (layer Edge.Cuts) (width 0.15))
-  (segment (start 70.8 150.45) (end 70.8 148.7) (width 0.13) (layer B.Cu) (net 1))
   (segment (start 70.8 148.7) (end 70.75 148.65) (width 0.13) (layer B.Cu) (net 1))
   (via (at 70.75 148.65) (size 0.8) (drill 0.5) (layers F.Cu B.Cu) (net 1))
   (segment (start 70.8 151.95) (end 70.8 150.45) (width 0.13) (layer F.Cu) (net 1))
   (via (at 70.8 150.45) (size 0.8) (drill 0.5) (layers F.Cu B.Cu) (net 1))
-  (segment (start 70.8 153.75) (end 70.8 151.95) (width 0.13) (layer B.Cu) (net 1))
   (via (at 70.8 151.95) (size 0.8) (drill 0.5) (layers F.Cu B.Cu) (net 1))
   (segment (start 70.8 155.5) (end 70.8 153.75) (width 0.13) (layer F.Cu) (net 1))
   (via (at 70.8 153.75) (size 0.8) (drill 0.5) (layers F.Cu B.Cu) (net 1))
-  (segment (start 70.8 157.5) (end 70.8 155.5) (width 0.13) (layer B.Cu) (net 1))
   (via (at 70.8 155.5) (size 0.8) (drill 0.5) (layers F.Cu B.Cu) (net 1))
   (segment (start 70.8 159.15) (end 70.8 157.5) (width 0.13) (layer F.Cu) (net 1))
   (via (at 70.8 157.5) (size 0.8) (drill 0.5) (layers F.Cu B.Cu) (net 1))
-  (segment (start 70.8 160.85) (end 70.8 159.15) (width 0.13) (layer B.Cu) (net 1))
   (via (at 70.8 159.15) (size 0.8) (drill 0.5) (layers F.Cu B.Cu) (net 1))
   (segment (start 70.8 162.55) (end 70.8 160.85) (width 0.13) (layer F.Cu) (net 1))
   (via (at 70.8 160.85) (size 0.8) (drill 0.5) (layers F.Cu B.Cu) (net 1))
-  (segment (start 70.8 163.334315) (end 70.8 162.55) (width 0.13) (layer B.Cu) (net 1))
   (via (at 70.8 162.55) (size 0.8) (drill 0.5) (layers F.Cu B.Cu) (net 1))
-  (segment (start 70.8 163.9) (end 70.8 163.334315) (width 0.13) (layer B.Cu) (net 1))
   (segment (start 70.8 165.4) (end 70.8 163.9) (width 0.13) (layer F.Cu) (net 1))
   (via (at 70.8 163.9) (size 0.8) (drill 0.5) (layers F.Cu B.Cu) (net 1))
   (via (at 70.8 165.4) (size 0.8) (drill 0.5) (layers F.Cu B.Cu) (net 1))
   (segment (start 67.6 165.4) (end 70.8 165.4) (width 0.13) (layer F.Cu) (net 1))
-  (segment (start 81.95 91.15) (end 84.65 91.15) (width 0.13) (layer B.Cu) (net 1))
   (via (at 84.65 91.15) (size 0.8) (drill 0.5) (layers F.Cu B.Cu) (net 1))
   (segment (start 79.85 91.15) (end 81.95 91.15) (width 0.13) (layer F.Cu) (net 1))
   (via (at 81.95 91.15) (size 0.8) (drill 0.5) (layers F.Cu B.Cu) (net 1))
-  (segment (start 79.85 89.15) (end 79.85 91.15) (width 0.13) (layer B.Cu) (net 1))
   (via (at 79.85 91.15) (size 0.8) (drill 0.5) (layers F.Cu B.Cu) (net 1))
   (segment (start 79.85 87.25) (end 79.85 89.15) (width 0.13) (layer F.Cu) (net 1))
   (via (at 79.85 89.15) (size 0.8) (drill 0.5) (layers F.Cu B.Cu) (net 1))
-  (segment (start 79.85 85.9) (end 79.85 87.25) (width 0.13) (layer B.Cu) (net 1))
   (via (at 79.85 87.25) (size 0.8) (drill 0.5) (layers F.Cu B.Cu) (net 1))
   (segment (start 82.2 85.9) (end 79.85 85.9) (width 0.13) (layer F.Cu) (net 1))
   (via (at 79.85 85.9) (size 0.8) (drill 0.5) (layers F.Cu B.Cu) (net 1))
-  (segment (start 84.75 85.9) (end 82.2 85.9) (width 0.13) (layer B.Cu) (net 1))
   (via (at 82.2 85.9) (size 0.8) (drill 0.5) (layers F.Cu B.Cu) (net 1))
   (segment (start 84.75 88.8) (end 84.75 85.9) (width 0.13) (layer F.Cu) (net 1))
@@
   (via (at 84.55 111.1) (size 0.8) (drill 0.5) (layers F.Cu B.Cu) (net 1))
   (via (at 81.1 111.15) (size 0.8) (drill 0.5) (layers F.Cu B.Cu) (net 1))
-  (segment (start 90.65 122.200004) (end 89.350004 122.200004) (width 0.13) (layer B.Cu) (net 1))
   (segment (start 87.95 122.2) (end 89.35 122.2) (width 0.13) (layer F.Cu) (net 1))
   (segment (start 89.350004 122.200004) (end 89.35 122.2) (width 0.13) (layer B.Cu) (net 1))
@@
   (segment (start 92.25 121) (end 92.25 119.35) (width 0.13) (layer F.Cu) (net 1))
   (via (at 92.25 119.35) (size 0.8) (drill 0.5) (layers F.Cu B.Cu) (net 1))
-  (segment (start 92.25 122.2) (end 92.25 121) (width 0.13) (layer B.Cu) (net 1))
   (via (at 92.25 121) (size 0.8) (drill 0.5) (layers F.Cu B.Cu) (net 1))
   (via (at 92.25 122.2) (size 0.8) (drill 0.5) (layers F.Cu B.Cu) (net 1))
-  (segment (start 87.95 120.9) (end 87.95 122.2) (width 0.13) (layer B.Cu) (net 1))
   (via (at 87.95 122.2) (size 0.8) (drill 0.5) (layers F.Cu B.Cu) (net 1))
   (segment (start 88 119.4) (end 88 120.85) (width 0.13) (layer F.Cu) (net 1))
@@
   (via (at 87.95 120.9) (size 0.8) (drill 0.5) (layers F.Cu B.Cu) (net 1))
   (via (at 88 119.4) (size 0.8) (drill 0.5) (layers F.Cu B.Cu) (net 1))
-  (segment (start 59.7 90.35) (end 61.9 90.35) (width 0.13) (layer B.Cu) (net 1))
   (via (at 61.9 90.35) (size 0.8) (drill 0.5) (layers F.Cu B.Cu) (net 1))
   (segment (start 58 90.35) (end 59.7 90.35) (width 0.13) (layer F.Cu) (net 1))
   (via (at 59.7 90.35) (size 0.8) (drill 0.5) (layers F.Cu B.Cu) (net 1))
-  (segment (start 58 88.9) (end 58 90.35) (width 0.13) (layer B.Cu) (net 1))
   (via (at 58 90.35) (size 0.8) (drill 0.5) (layers F.Cu B.Cu) (net 1))
   (segment (start 57.95 87.3) (end 57.95 88.85) (width 0.13) (layer F.Cu) (net 1))
   (segment (start 57.95 88.85) (end 58 88.9) (width 0.13) (layer F.Cu) (net 1))
   (via (at 58 88.9) (size 0.8) (drill 0.5) (layers F.Cu B.Cu) (net 1))
-  (segment (start 57.95 85.65) (end 57.95 87.3) (width 0.13) (layer B.Cu) (net 1))
   (via (at 57.95 87.3) (size 0.8) (drill 0.5) (layers F.Cu B.Cu) (net 1))
   (segment (start 60.05 85.7) (end 58 85.7) (width 0.13) (layer F.Cu) (net 1))
   (segment (start 58 85.7) (end 57.95 85.65) (width 0.13) (layer F.Cu) (net 1))
   (via (at 57.95 85.65) (size 0.8) (drill 0.5) (layers F.Cu B.Cu) (net 1))
-  (segment (start 61.9 85.7) (end 60.05 85.7) (width 0.13) (layer B.Cu) (net 1))
   (via (at 60.05 85.7) (size 0.8) (drill 0.5) (layers F.Cu B.Cu) (net 1))
   (segment (start 61.9 88.05) (end 61.9 86.282234) (width 0.13) (layer F.Cu) (net 1))
@@
   (segment (start 70.3 120.3) (end 70.3 119.2) (width 0.13) (layer F.Cu) (net 1))
   (via (at 70.3 119.2) (size 0.8) (drill 0.5) (layers F.Cu B.Cu) (net 1))
-  (segment (start 70.3 121.2) (end 70.3 120.3) (width 0.13) (layer B.Cu) (net 1))
   (via (at 70.3 120.3) (size 0.8) (drill 0.5) (layers F.Cu B.Cu) (net 1))
   (segment (start 68.85 121.2) (end 70.3 121.2) (width 0.13) (layer F.Cu) (net 1))
   (via (at 70.3 121.2) (size 0.8) (drill 0.5) (layers F.Cu B.Cu) (net 1))
-  (segment (start 67.8 121.2) (end 68.85 121.2) (width 0.13) (layer B.Cu) (net 1))
   (via (at 68.85 121.2) (size 0.8) (drill 0.5) (layers F.Cu B.Cu) (net 1))
   (segment (start 66.65 121.15) (end 67.75 121.15) (width 0.13) (layer F.Cu) (net 1))
   (segment (start 67.75 121.15) (end 67.8 121.2) (width 0.13) (layer F.Cu) (net 1))
   (via (at 67.8 121.2) (size 0.8) (drill 0.5) (layers F.Cu B.Cu) (net 1))
-  (segment (start 66.65 120.2) (end 66.65 121.15) (width 0.13) (layer B.Cu) (net 1))
   (via (at 66.65 121.15) (size 0.8) (drill 0.5) (layers F.Cu B.Cu) (net 1))
   (segment (start 66.65 119.2) (end 66.65 120.2) (width 0.13) (layer F.Cu) (net 1))
@@
   (segment (start 81.75 114.3) (end 81.75 114.6) (width 0.13) (layer F.Cu) (net 6))
   (via (at 81.75 114.6) (size 0.8) (drill 0.5) (layers F.Cu B.Cu) (net 6))
-  (segment (start 67.6 90.25) (end 65.1 90.25) (width 0.13) (layer B.Cu) (net 8))
   (via (at 65.1 90.25) (size 0.8) (drill 0.5) (layers F.Cu B.Cu) (net 8))
   (segment (start 69.6 90.25) (end 67.6 90.25) (width 0.13) (layer F.Cu) (net 8))
   (via (at 67.6 90.25) (size 0.8) (drill 0.5) (layers F.Cu B.Cu) (net 8))
-  (segment (start 69.6 88.75) (end 69.6 90.25) (width 0.13) (layer B.Cu) (net 8))
   (via (at 69.6 90.25) (size 0.8) (drill 0.5) (layers F.Cu B.Cu) (net 8))
   (segment (start 69.6 87.15) (end 69.6 88.75) (width 0.13) (layer F.Cu) (net 8))
   (via (at 69.6 88.75) (size 0.8) (drill 0.5) (layers F.Cu B.Cu) (net 8))
-  (segment (start 69.6 85.75) (end 69.6 87.15) (width 0.13) (layer B.Cu) (net 8))
   (via (at 69.6 87.15) (size 0.8) (drill 0.5) (layers F.Cu B.Cu) (net 8))
   (segment (start 67.65 85.75) (end 69.6 85.75) (width 0.13) (layer F.Cu) (net 8))
   (via (at 69.6 85.75) (size 0.8) (drill 0.5) (layers F.Cu B.Cu) (net 8))
-  (segment (start 65.1 85.75) (end 67.65 85.75) (width 0.13) (layer B.Cu) (net 8))
   (via (at 67.65 85.75) (size 0.8) (drill 0.5) (layers F.Cu B.Cu) (net 8))
   (segment (start 65.1 88.05) (end 65.1 85.75) (width 0.13) (layer F.Cu) (net 8))
@@
       )
     )
+  )
+  (zone (net 1) (net_name Earth) (layer F.Mask) (hatch edge 0.508)
+    (connect_pads (clearance 0.2))
+    (min_thickness 0.254)
+    (fill yes (arc_segments 16) (thermal_gap 0.508) (thermal_bridge_width 0.508))
+    (polygon
+      (pts
+        (xy 86.15 118.7) (xy 94.05 118.7) (xy 94.05 123.1) (xy 86.15 123.1)
+      )
+    )
+  )
+  (zone (net 1) (net_name Earth) (layer F.Cu) (hatch edge 0.508)
+    (connect_pads yes (clearance 0.2))
+    (min_thickness 0.254)
+    (fill yes (arc_segments 16) (thermal_gap 0.508) (thermal_bridge_width 0.508))
+    (polygon
+      (pts
+        (xy 50.45 37.35) (xy 54.25 37.35) (xy 54.25 47.7) (xy 50.45 47.7)
+      )
+    )

Commit message: donno what I'm committing
Parts:
- removed C7, C8: 0.01uF 50V, Capacitors_SMD:C_0603
- removed D8: D_Small, Diodes_SMD:D_SMA
- removed Q2: SQJ459EP, Dizzy:SQJ459EP
- added C1: 20uF 50V, Capacitors_SMD:C_1210, F.Cu at (65.1, 154.7)
- added C4: 20uF 50V, Capacitors_SMD:C_1210, F.Cu at (76.1, 158.8)
- added C5: 20uF 50V, Capacitors_SMD:C_1210, F.Cu at (76.1, 162.2)
- added R2: 47K, Resistors_SMD:R_0603, F.Cu at (53.6, 141.7)
- C22: value 20uF -> 20uF 50V; footprint Capacitors_SMD:C_1812 -> Capacitors_SMD:C_1210
- D5: footprint Diodes_SMD:D_SMA -> Diodes_SMD:D_SMC
- Q1: value BSS123W -> SQM120P04-04L; footprint TO_SOT_Packages_SMD:SOT-323_SC-70 -> TO_SOT_Packages_SMD:TO-263-2
- R1: value 1K -> 47K
- R14: value 62k 1% -> 30K 1%
- U1: value LM2678-3.3V -> AP1501A-3.3V; footprint Dizzy:14-VSON -> TO_SOT_Packages_SMD:TO-263-5_TabPin3
- U10: value LTC2954-1 -> LTC2954-2
- U2: value LM2678-12V -> AP1501A-12V; footprint Dizzy:14-VSON -> TO_SOT_Packages_SMD:TO-263-5_TabPin3
- moved C13 25.0 mm to (76.5, 89.2), turned to 180 degrees
- moved C28 24.7 mm to (55.9, 88.9), turned to 180 degrees
- moved C29 23.4 mm to (76.5, 94.0), turned to 180 degrees
- moved C12 22.6 mm to (55.9, 93.7), turned to 180 degrees
- moved Q1 16.4 mm to (71.3, 141.7), turned to 0 degrees
- moved D4 9.31 mm to (59.1, 129.2)
- moved C22 8.75 mm to (65.1, 150.8)
- moved D3 8.49 mm to (81.0, 128.0)
- moved J9 8.28 mm to (80.9, 80.0)
- moved L2 7.99 mm to (85.1, 91.9), turned to 90 degrees
- moved L1 6.97 mm to (65.0, 91.9), turned to 90 degrees
- moved J8 6.01 mm to (60.8, 81.0)
- moved U2 5.50 mm to (79.5, 113.3), turned to 270 degrees
- moved U1 4.96 mm to (59.0, 113.3), turned to 270 degrees
- moved D1 4.87 mm to (58.2, 101.1), turned to 180 degrees
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- renumbered C19 to 0.1, C20 to 0.1, C21 to 0.1, C23 to 0.1, C24 to 0.1, C25 to 0.1, C26 to 0.1
Connections:
- C10 pad 1: Earth -> Net-(C10-Pad1)
- C10 pad 2: Net-(C10-Pad2) -> Earth
- C2 pad 1: Earth -> Net-(C10-Pad1)
- C2 pad 2: Net-(C10-Pad2) -> Earth
- C3 pad 1: Earth -> Net-(C3-Pad1)
- C3 pad 2: Net-(C3-Pad2) -> Earth
- C9 pad 1: Earth -> Net-(C3-Pad1)
- C9 pad 2: Net-(C3-Pad2) -> Earth
- D1 pad 1: Net-(C7-Pad2) -> Net-(D1-Pad1)
- D2 pad 1: Net-(C8-Pad2) -> Net-(D2-Pad1)
- D3 pad 1: Net-(C3-Pad2) -> Net-(C3-Pad1)
- D4 pad 1: Net-(C10-Pad2) -> Net-(C10-Pad1)
- L1 pad 1: Net-(C7-Pad2) -> Net-(D1-Pad1)
- L2 pad 1: Net-(C8-Pad2) -> Net-(D2-Pad1)
- Q1 pad 1: PWR_EN -> Net-(Q1-Pad1)
- Q1 pad 2: Earth -> Net-(Q1-Pad2)
- Q1 pad 3: Net-(Q1-Pad3) -> +BATT
- R1 pad 1: Net-(Q1-Pad3) -> PWR_EN
- U1 pad 1: (no net) -> Net-(C10-Pad1)
- U1 pad 2: Net-(C10-Pad2) -> Net-(D1-Pad1)
- U1 pad 3: Net-(C10-Pad2) -> Earth
- U1 pad 4: Net-(C7-Pad1) -> 3.3V
- U1 pad 5: (no net) -> PWR_EN
- U2 pad 1: (no net) -> Net-(C3-Pad1)
- U2 pad 2: Net-(C3-Pad2) -> Net-(D2-Pad1)
- U2 pad 3: Net-(C3-Pad2) -> Earth
- U2 pad 4: Net-(C8-Pad1) -> 12V
- U2 pad 5: (no net) -> PWR_EN
- U6 pad 5: Net-(Q2-Pad3) -> Net-(Q1-Pad2)
Routing:
- net Earth: track 97.0 -> 145.4 mm, vias 91 -> 87
- net PWR_EN: track 169.7 -> 130.4 mm, vias 2 -> 4
- net Net-(Q1-Pad3): track 22.0 -> 0.00 mm, vias 2 -> 0
- net 3.3V: track 37.2 -> 51.4 mm, vias 28 -> 24
- net Net-(Q1-Pad1): track 0.00 -> 13.1 mm, vias 0 -> 2
- net 12V: track 11.1 -> 22.8 mm
- net Net-(C7-Pad1): track 9.15 -> 0.00 mm, vias 2 -> 0
- net Net-(C8-Pad1): track 8.90 -> 0.00 mm, vias 2 -> 0
- net Net-(C8-Pad2): track 4.12 -> 0.00 mm
- net Net-(C7-Pad2): track 3.45 -> 0.00 mm
- net Net-(R17-Pad1): track 105.9 -> 109.1 mm
- net +BATT: track 114.6 -> 115.9 mm
- added copper zone on F.Cu, net Net-(C10-Pad1)
- added copper zone on F.Cu, net Net-(C3-Pad1)
- added copper zone on F.Cu, net Net-(D1-Pad1)
- added copper zone on F.Cu, net Net-(D2-Pad1)
- added copper zone on F.Cu, net Net-(Q1-Pad2)
- removed copper zone on F.Cu, net Net-(C10-Pad2)
- removed copper zone on F.Cu, net Net-(C3-Pad2)
- removed copper zone on F.Cu, net Net-(C7-Pad2)
- removed copper zone on F.Cu, net Net-(C8-Pad2)
- removed copper zone on F.Cu, net Net-(Q2-Pad3)
